Commit message: simulation

File: rotors_description/urdf/multirotor_base.xacro (robot description, xacro)
@@ -69,5 +69,5 @@
         <robotNamespace>${robot_namespace}</robotNamespace>
         <linkName>${robot_namespace}/base_link</linkName>
-        <rotorVelocitySlowdownSim>${rotor_velocity_slowdown_sim}</rotorVelocitySlowdownSim>
+        <rotorVelocitySlowdownSim>${rotor_velocity_slowdown_thrust}</rotorVelocitySlowdownSim>
       </plugin>
     </gazebo>
@@ -86,5 +86,5 @@
     <link name="${robot_namespace}/rotor_${motor_number}">
       <inertial>
-        <mass value="${mass_rotor}" /> <!-- [kg] -->
+        <mass value="${mass_rotor_thrust}" /> <!-- [kg] -->
         <xacro:insert_block name="inertia" />
       </inertial>
@@ -97,5 +97,5 @@
           </xacro:if>
           <xacro:unless value="${use_own_mesh}">
-            <mesh filename="package://rotors_description/meshes/propeller_${direction}.dae"
+            <mesh filename="package://rotors_description/meshes/geranos_prop_${direction}.dae"
               scale="${radius_rotor} ${radius_rotor} ${radius_rotor}" /> <!-- The propeller meshes have a radius of 1m -->
             <!-- <box size="${2*radius_rotor} 0.01 0.005"/> -->
@@ -125,5 +125,5 @@
         <rollingMomentCoefficient>${rolling_moment_coefficient}</rollingMomentCoefficient>
         <motorSpeedPubTopic>motor_speed/${motor_number}</motorSpeedPubTopic>
-        <rotorVelocitySlowdownSim>${rotor_velocity_slowdown_sim}</rotorVelocitySlowdownSim>
+        <rotorVelocitySlowdownSim>${rotor_velocity_slowdown_thrust}</rotorVelocitySlowdownSim>
       </plugin>
     </gazebo>

Commit message: Bug in MultirotorBase

File: rotors_description/urdf/multirotor_base.xacro (robot description, xacro)
@@ -37,5 +37,5 @@
     <!-- origin -->
     <joint name="${robot_namespace}/base_joint" type="fixed">
-      <origin xyz="0.001 0 0" rpy="0 0 0" />
+      <origin xyz="0 0 0" rpy="0 0 0" />
       <parent link="${robot_namespace}/base_link" />
       <child link="${robot_namespace}/base_link_inertia" />
