Commit message: simulation

File: rotors_description/urdf/geranos.xacro (robot description, xacro)
@@ -8,5 +8,5 @@
   <xacro:property name="use_mesh_file" value="true" />
   <xacro:property name="mesh_file" value="package://rotors_description/meshes/geranos_simple.dae" />
-  <xacro:property name="mass" value="4.7" /> <!-- [kg] --> <!-- still to be determined -->
+  <xacro:property name="mass" value="5.0" /> <!-- [kg] --> <!-- still to be determined -->
   <xacro:property name="body_width" value="0.820" /> <!-- [m] -->
   <xacro:property name="half_body_width_long" value="0.44" /> <!-- [m] -->
@@ -31,5 +31,5 @@
   <!-- Property Blocks -->
   <xacro:property name="body_inertia"> <!-- still to be determined -->
-    <inertia ixx="1.5" ixy="0.0" ixz="0.0" iyy="1.5" iyz="0.0" izz="1.5" /> <!-- [kg.m^2] [kg.m^2] [kg.m^2] [kg.m^2] [kg.m^2] [kg.m^2] -->
+    <inertia ixx="0.06" ixy="0.0" ixz="0.0" iyy="0.10" iyz="0.0" izz="0.15" /> <!-- [kg.m^2] [kg.m^2] [kg.m^2] [kg.m^2] [kg.m^2] [kg.m^2] -->
   </xacro:property>
   <!-- inertia of a single rotor, assuming it is a cuboid. Height=3mm, width=15mm -->
@@ -147,4 +147,24 @@
     time_constant_down="${time_constant_down}"
     max_rot_velocity="${max_rot_velocity}"
+    motor_number="6"
+    rotor_drag_coefficient="${rotor_drag_coefficient}"
+    rolling_moment_coefficient="${rolling_moment_coefficient}"
+    color="Blue"
+    use_own_mesh="false"
+    mesh="">
+    <origin xyz="0.465  0 ${rotor_offset_direction}" rpy="0 -0.698132 0" />
+    <xacro:insert_block name="rotor_inertia_direction" />
+  </xacro:vertical_rotor>
+  <xacro:vertical_rotor robot_namespace="${namespace}"
+    suffix="direciton_left"
+    direction="direction"
+    motor_constant="${motor_constant}"
+    moment_constant="${moment_constant}"
+    parent="${namespace}/base_link"
+    mass_rotor="${mass_rotor_direction}"
+    radius_rotor="${radius_rotor_direction}"
+    time_constant_up="${time_constant_up}"
+    time_constant_down="${time_constant_down}"
+    max_rot_velocity="${max_rot_velocity}"
     motor_number="4"
     rotor_drag_coefficient="${rotor_drag_coefficient}"
@@ -153,9 +173,9 @@
     use_own_mesh="false"
     mesh="">
-    <origin xyz="0.465  0 ${rotor_offset_direction}" rpy="0 -0.698132 0" />
-    <xacro:insert_block name="rotor_inertia_direction" />
-  </xacro:vertical_rotor>
-  <xacro:vertical_rotor robot_namespace="${namespace}"
-    suffix="direciton_left"
+    <origin xyz="-0.452 0 0.28" rpy="0 0.698132 0" />
+    <xacro:insert_block name="rotor_inertia_direction" />
+  </xacro:vertical_rotor>
+  <xacro:vertical_rotor robot_namespace="${namespace}"
+    suffix="direction_front"
     direction="direction"
     motor_constant="${motor_constant}"
@@ -173,24 +193,4 @@
     use_own_mesh="false"
     mesh="">
-    <origin xyz="-0.452 0 0.28" rpy="0 0.698132 0" />
-    <xacro:insert_block name="rotor_inertia_direction" />
-  </xacro:vertical_rotor>
-  <xacro:vertical_rotor robot_namespace="${namespace}"
-    suffix="direction_front"
-    direction="direction"
-    motor_constant="${motor_constant}"
-    moment_constant="${moment_constant}"
-    parent="${namespace}/base_link"
-    mass_rotor="${mass_rotor_direction}"
-    radius_rotor="${radius_rotor_direction}"
-    time_constant_up="${time_constant_up}"
-    time_constant_down="${time_constant_down}"
-    max_rot_velocity="${max_rot_velocity}"
-    motor_number="6"
-    rotor_drag_coefficient="${rotor_drag_coefficient}"
-    rolling_moment_coefficient="${rolling_moment_coefficient}"
-    color="Blue"
-    use_own_mesh="false"
-    mesh="">
     <origin xyz="0 0.365  ${rotor_offset_direction}" rpy="0.698132 0 0" />
     <xacro:insert_block name="rotor_inertia_direction" />
@@ -216,4 +216,80 @@
     <xacro:insert_block name="rotor_inertia_direction" />
   </xacro:vertical_rotor>
+   <gazebo>
+    <plugin name="mavlink_interface" filename="librotors_gazebo_mavlink_interface.so">
+      <robotNamespace>${namespace}</robotNamespace>
+      <imu_rate>102</imu_rate>
+      <imuSubTopic>/imu</imuSubTopic>
+      <mavlink_addr>INADDR_ANY</mavlink_addr>
+      <mavlink_udp_port>14560</mavlink_udp_port>
+      <motorSpeedCommandPubTopic>/gazebo/command/motor_speed</motorSpeedCommandPubTopic>
+      <control_channels>
+        <channel name="rotor0">
+          <input_index>0</input_index>
+          <input_offset>0</input_offset>
+          <input_scaling>${max_rot_velocity}</input_scaling>
+          <zero_position_disarmed>0</zero_position_disarmed>
+          <zero_position_armed>100</zero_position_armed>
+          <joint_control_type>velocity</joint_control_type>
+        </channel>
+        <channel name="rotor1">
+          <input_index>1</input_index>
+          <input_offset>0</input_offset>
+          <input_scaling>${max_rot_velocity}</input_scaling>
+          <zero_position_disarmed>0</zero_position_disarmed>
+          <zero_position_armed>100</zero_position_armed>
+          <joint_control_type>velocity</joint_control_type>
+        </channel>
+        <channel name="rotor2">
+          <input_index>2</input_index>
+          <input_offset>0</input_offset>
+          <input_scaling>${max_rot_velocity}</input_scaling>
+          <zero_position_disarmed>0</zero_position_disarmed>
+          <zero_position_armed>100</zero_position_armed>
+          <joint_control_type>velocity</joint_control_type>
+        </channel>
+        <channel name="rotor3">
+          <input_index>3</input_index>
+          <input_offset>0</input_offset>
+          <input_scaling>${max_rot_velocity}</input_scaling>
+          <zero_position_disarmed>0</zero_position_disarmed>
+          <zero_position_armed>100</zero_position_armed>
+          <joint_control_type>velocity</joint_control_type>
+        </channel>
+        <channel name="rotor4">
+          <input_index>4</input_index>
+          <input_offset>0</input_offset>
+          <input_scaling>${max_rot_velocity}</input_scaling>
+          <zero_position_disarmed>0</zero_position_disarmed>
+          <zero_position_armed>100</zero_position_armed>
+          <joint_control_type>velocity</joint_control_type>
+        </channel>
+        <channel name="rotor5">
+          <input_index>5</input_index>
+          <input_offset>0</input_offset>
+          <input_scaling>${max_rot_velocity}</input_scaling>
+          <zero_position_disarmed>0</zero_position_disarmed>
+          <zero_position_armed>100</zero_position_armed>
+          <joint_control_type>velocity</joint_control_type>
+        </channel>
+         <channel name="rotor6">
+          <input_index>6</input_index>
+          <input_offset>0</input_offset>
+          <input_scaling>${max_rot_velocity}</input_scaling>
+          <zero_position_disarmed>0</zero_position_disarmed>
+          <zero_position_armed>100</zero_position_armed>
+          <joint_control_type>velocity</joint_control_type>
+        </channel>
+        <channel name="rotor7">
+          <input_index>7</input_index>
+          <input_offset>0</input_offset>
+          <input_scaling>${max_rot_velocity}</input_scaling>
+          <zero_position_disarmed>0</zero_position_disarmed>
+          <zero_position_armed>100</zero_position_armed>
+          <joint_control_type>velocity</joint_control_type>
+        </channel>
+      </control_channels>
+    </plugin>
+  </gazebo>
 </robot>
 <!-- add channel from omav.xacro-->

Commit message: Corrected Rotor numbering

File: rotors_description/urdf/geranos.xacro (robot description, xacro)
@@ -21,5 +21,5 @@
   <xacro:property name="rotor_offset_direction" value="0.27" /> <!-- [m] --> <!-- still to be determined -->
   <xacro:property name="radius_rotor_thrust" value="1" /> <!-- [m] --> <!-- radius or durchmesser -->
-  <xacro:property name="radius_rotor_direction" value="0.5" /> <!-- [m] --> <!-- radius or durchmesser -->
+  <xacro:property name="radius_rotor_direction" value="1" /> <!-- [m] --> <!-- radius or durchmesser -->
   <xacro:property name="motor_constant" value="8.54858e-06" /> <!-- [kg.m/s^2] -->  <!-- still to be determined -->
   <xacro:property name="moment_constant" value="0.016" /> <!-- [m] --> <!-- still to be determined -->
@@ -66,5 +66,5 @@
     time_constant_down="${time_constant_down}"
     max_rot_velocity="${max_rot_velocity}"
-    motor_number="0"
+    motor_number="2"
     rotor_drag_coefficient="${rotor_drag_coefficient}"
     rolling_moment_coefficient="${rolling_moment_coefficient}"
@@ -87,4 +87,24 @@
     time_constant_down="${time_constant_down}"
     max_rot_velocity="${max_rot_velocity}"
+    motor_number="0"
+    rotor_drag_coefficient="${rotor_drag_coefficient}"
+    rolling_moment_coefficient="${rolling_moment_coefficient}"
+    color="Red"
+    use_own_mesh="false"
+    mesh="">
+    <origin xyz="-${half_body_width_long} -${half_body_width_short} ${rotor_offset_thrust}" rpy="0 0 0" />
+    <xacro:insert_block name="rotor_inertia_thrust" />
+  </xacro:vertical_rotor>
+  <xacro:vertical_rotor robot_namespace="${namespace}"
+    suffix="back_right"
+    direction="thrust"
+    motor_constant="${motor_constant}"
+    moment_constant="${moment_constant}"
+    parent="${namespace}/base_link"
+    mass_rotor="${mass_rotor_thrust}"
+    radius_rotor="${radius_rotor_thrust}"
+    time_constant_up="${time_constant_up}"
+    time_constant_down="${time_constant_down}"
+    max_rot_velocity="${max_rot_velocity}"
     motor_number="1"
     rotor_drag_coefficient="${rotor_drag_coefficient}"
@@ -93,5 +113,5 @@
     use_own_mesh="false"
     mesh="">
-    <origin xyz="-${half_body_width_long} -${half_body_width_short} ${rotor_offset_thrust}" rpy="0 0 0" />
+    <origin xyz="-${half_body_width_long} ${half_body_width_short} ${rotor_offset_thrust}" rpy="0 0 0" />
     <xacro:insert_block name="rotor_inertia_thrust" />
   </xacro:vertical_rotor>
@@ -107,24 +127,4 @@
     time_constant_down="${time_constant_down}"
     max_rot_velocity="${max_rot_velocity}"
-    motor_number="2"
-    rotor_drag_coefficient="${rotor_drag_coefficient}"
-    rolling_moment_coefficient="${rolling_moment_coefficient}"
-    color="Red"
-    use_own_mesh="false"
-    mesh="">
-    <origin xyz="-${half_body_width_long} ${half_body_width_short} ${rotor_offset_thrust}" rpy="0 0 0" />
-    <xacro:insert_block name="rotor_inertia_thrust" />
-  </xacro:vertical_rotor>
-  <xacro:vertical_rotor robot_namespace="${namespace}"
-    suffix="back_right"
-    direction="thrust"
-    motor_constant="${motor_constant}"
-    moment_constant="${moment_constant}"
-    parent="${namespace}/base_link"
-    mass_rotor="${mass_rotor_thrust}"
-    radius_rotor="${radius_rotor_thrust}"
-    time_constant_up="${time_constant_up}"
-    time_constant_down="${time_constant_down}"
-    max_rot_velocity="${max_rot_velocity}"
     motor_number="3"
     rotor_drag_coefficient="${rotor_drag_coefficient}"
@@ -137,4 +137,44 @@
   </xacro:vertical_rotor>
 <xacro:vertical_rotor robot_namespace="${namespace}"
+    suffix="direction_front"
+    direction="direction"
+    motor_constant="${motor_constant}"
+    moment_constant="${moment_constant}"
+    parent="${namespace}/base_link"
+    mass_rotor="${mass_rotor_direction}"
+    radius_rotor="${radius_rotor_direction}"
+    time_constant_up="${time_constant_up}"
+    time_constant_down="${time_constant_down}"
+    max_rot_velocity="${max_rot_velocity}"
+    motor_number="6"
+    rotor_drag_coefficient="${rotor_drag_coefficient}"
+    rolling_moment_coefficient="${rolling_moment_coefficient}"
+    color="Blue"
+    use_own_mesh="false"
+    mesh="">
+    <origin xyz="0.465  0 ${rotor_offset_direction}" rpy="0 -0.698132 0" />
+    <xacro:insert_block name="rotor_inertia_direction" />
+  </xacro:vertical_rotor>
+  <xacro:vertical_rotor robot_namespace="${namespace}"
+    suffix="direciton_back"
+    direction="direction"
+    motor_constant="${motor_constant}"
+    moment_constant="${moment_constant}"
+    parent="${namespace}/base_link"
+    mass_rotor="${mass_rotor_direction}"
+    radius_rotor="${radius_rotor_direction}"
+    time_constant_up="${time_constant_up}"
+    time_constant_down="${time_constant_down}"
+    max_rot_velocity="${max_rot_velocity}"
+    motor_number="4"
+    rotor_drag_coefficient="${rotor_drag_coefficient}"
+    rolling_moment_coefficient="${rolling_moment_coefficient}"
+    color="Blue"
+    use_own_mesh="false"
+    mesh="">
+    <origin xyz="-0.452 0 0.28" rpy="0 0.698132 0" />
+    <xacro:insert_block name="rotor_inertia_direction" />
+  </xacro:vertical_rotor>
+  <xacro:vertical_rotor robot_namespace="${namespace}"
     suffix="direction_right"
     direction="direction"
@@ -147,24 +187,4 @@
     time_constant_down="${time_constant_down}"
     max_rot_velocity="${max_rot_velocity}"
-    motor_number="4"
-    rotor_drag_coefficient="${rotor_drag_coefficient}"
-    rolling_moment_coefficient="${rolling_moment_coefficient}"
-    color="Blue"
-    use_own_mesh="false"
-    mesh="">
-    <origin xyz="0.465  0 ${rotor_offset_direction}" rpy="0 -0.698132 0" />
-    <xacro:insert_block name="rotor_inertia_direction" />
-  </xacro:vertical_rotor>
-  <xacro:vertical_rotor robot_namespace="${namespace}"
-    suffix="direciton_left"
-    direction="direction"
-    motor_constant="${motor_constant}"
-    moment_constant="${moment_constant}"
-    parent="${namespace}/base_link"
-    mass_rotor="${mass_rotor_direction}"
-    radius_rotor="${radius_rotor_direction}"
-    time_constant_up="${time_constant_up}"
-    time_constant_down="${time_constant_down}"
-    max_rot_velocity="${max_rot_velocity}"
     motor_number="5"
     rotor_drag_coefficient="${rotor_drag_coefficient}"
@@ -173,29 +193,9 @@
     use_own_mesh="false"
     mesh="">
-    <origin xyz="-0.452 0 0.28" rpy="0 0.698132 0" />
-    <xacro:insert_block name="rotor_inertia_direction" />
-  </xacro:vertical_rotor>
-  <xacro:vertical_rotor robot_namespace="${namespace}"
-    suffix="direction_front"
-    direction="direction"
-    motor_constant="${motor_constant}"
-    moment_constant="${moment_constant}"
-    parent="${namespace}/base_link"
-    mass_rotor="${mass_rotor_direction}"
-    radius_rotor="${radius_rotor_direction}"
-    time_constant_up="${time_constant_up}"
-    time_constant_down="${time_constant_down}"
-    max_rot_velocity="${max_rot_velocity}"
-    motor_number="6"
-    rotor_drag_coefficient="${rotor_drag_coefficient}"
-    rolling_moment_coefficient="${rolling_moment_coefficient}"
-    color="Blue"
-    use_own_mesh="false"
-    mesh="">
     <origin xyz="0 0.365  ${rotor_offset_direction}" rpy="0.698132 0 0" />
     <xacro:insert_block name="rotor_inertia_direction" />
   </xacro:vertical_rotor>
   <xacro:vertical_rotor robot_namespace="${namespace}"
-    suffix="direction_back"
+    suffix="direction_left"
     direction="direction"
     motor_constant="${motor_constant}"

Commit message: Corrected Position Values for Rotors

File: rotors_description/urdf/geranos.xacro (robot description, xacro)
@@ -10,6 +10,8 @@
   <xacro:property name="mass" value="5.0" /> <!-- [kg] --> <!-- still to be determined -->
   <xacro:property name="body_width" value="0.820" /> <!-- [m] -->
-  <xacro:property name="half_body_width_long" value="0.44" /> <!-- [m] -->
-  <xacro:property name="half_body_width_short" value="0.41" /> <!-- [m] -->
+  <xacro:property name="big_rotor_x" value="0.44017" /> <!-- [m] -->
+  <xacro:property name="big_rotor_y" value="0.4098" /> <!-- [m] -->
+  <xacro:property name="small_rotor_x" value="0.46506" /> <!-- [m] -->
+  <xacro:property name="small_rotor_y" value="0.36506" /> <!-- [m] -->
   <xacro:property name="half_body_width" value="0.3" /> <!-- [m] -->
   <xacro:property name="side_length_one" value="0.2" /> <!-- [m] -->
@@ -72,5 +74,5 @@
     use_own_mesh="false"
     mesh="">
-    <origin xyz="${half_body_width_long} ${half_body_width_short} ${rotor_offset_thrust}" rpy="0 0 0" />
+    <origin xyz="${big_rotor_x} ${big_rotor_y} ${rotor_offset_thrust}" rpy="0 0 0" />
     <xacro:insert_block name="rotor_inertia_thrust" />
   </xacro:vertical_rotor>
@@ -93,5 +95,5 @@
     use_own_mesh="false"
     mesh="">
-    <origin xyz="-${half_body_width_long} -${half_body_width_short} ${rotor_offset_thrust}" rpy="0 0 0" />
+    <origin xyz="-${big_rotor_x} -${big_rotor_y} ${rotor_offset_thrust}" rpy="0 0 0" />
     <xacro:insert_block name="rotor_inertia_thrust" />
   </xacro:vertical_rotor>
@@ -113,5 +115,5 @@
     use_own_mesh="false"
     mesh="">
-    <origin xyz="-${half_body_width_long} ${half_body_width_short} ${rotor_offset_thrust}" rpy="0 0 0" />
+    <origin xyz="-${big_rotor_x} ${big_rotor_y} ${rotor_offset_thrust}" rpy="0 0 0" />
     <xacro:insert_block name="rotor_inertia_thrust" />
   </xacro:vertical_rotor>
@@ -133,5 +135,5 @@
     use_own_mesh="false"
     mesh="">
-    <origin xyz="${half_body_width_long} -${half_body_width_short} ${rotor_offset_thrust}" rpy="0 0 0" />
+    <origin xyz="${big_rotor_x} -${big_rotor_y} ${rotor_offset_thrust}" rpy="0 0 0" />
     <xacro:insert_block name="rotor_inertia_thrust" />
   </xacro:vertical_rotor>
@@ -153,5 +155,5 @@
     use_own_mesh="false"
     mesh="">
-    <origin xyz="0.465  0 ${rotor_offset_direction}" rpy="0 -0.698132 0" />
+    <origin xyz="${small_rotor_x}  0 ${rotor_offset_direction}" rpy="0 -0.698132 0" />
     <xacro:insert_block name="rotor_inertia_direction" />
   </xacro:vertical_rotor>
@@ -173,5 +175,5 @@
     use_own_mesh="false"
     mesh="">
-    <origin xyz="-0.452 0 0.28" rpy="0 0.698132 0" />
+    <origin xyz="-${small_rotor_x} 0 ${rotor_offset_direction}" rpy="0 0.698132 0" />
     <xacro:insert_block name="rotor_inertia_direction" />
   </xacro:vertical_rotor>
@@ -193,5 +195,5 @@
     use_own_mesh="false"
     mesh="">
-    <origin xyz="0 0.365  ${rotor_offset_direction}" rpy="0.698132 0 0" />
+    <origin xyz="0 ${small_rotor_y}  ${rotor_offset_direction}" rpy="0.698132 0 0" />
     <xacro:insert_block name="rotor_inertia_direction" />
   </xacro:vertical_rotor>
@@ -213,5 +215,5 @@
     use_own_mesh="false"
     mesh="">
-    <origin xyz="0 -0.365  ${rotor_offset_direction}" rpy="-0.698132 0 0" />
+    <origin xyz="0 -${small_rotor_y}  ${rotor_offset_direction}" rpy="-0.698132 0 0" />
     <xacro:insert_block name="rotor_inertia_direction" />
   </xacro:vertical_rotor>
