Commit message: max_rotor_velocity increased and radius_rotor defined

File: rotors_description/urdf/geranos.xacro (robot description, xacro)
@@ -10,5 +10,5 @@
   <xacro:property name="mass" value="5.0" /> <!-- [kg] --> <!-- still to be determined -->
   <xacro:property name="body_width" value="0.820" /> <!-- [m] -->
-  <xacro:property name="big_rotor_x" value="0.44017" /> <!-- [m] -->
+   <xacro:property name="big_rotor_x" value="0.44017" /> <!-- [m] -->
   <xacro:property name="big_rotor_y" value="0.4098" /> <!-- [m] -->
   <xacro:property name="small_rotor_x" value="0.46506" /> <!-- [m] -->
@@ -22,11 +22,14 @@
   <xacro:property name="rotor_offset_thrust" value="0.13" /> <!-- [m] --> <!-- still to be determined -->
   <xacro:property name="rotor_offset_direction" value="0.27" /> <!-- [m] --> <!-- still to be determined -->
-  <xacro:property name="radius_rotor_thrust" value="1" /> <!-- [m] --> <!-- radius or durchmesser -->
-  <xacro:property name="radius_rotor_direction" value="1" /> <!-- [m] --> <!-- radius or durchmesser -->
+  <xacro:property name="radius_rotor_thrust_simulation" value="1" /> <!-- [m] --> <!-- radius or durchmesser -->
+  <xacro:property name="radius_rotor_direction_simulation" value="1" /> <!-- [m] --> <!-- radius or durchmesser -->
+  <xacro:property name="radius_rotor_thrust_meter" value="0.2286" /> <!-- [m] --> <!-- radius -->
+  <xacro:property name="radius_rotor_direction_meter" value="0.06477" /> <!-- [m] --> <!-- radius -->
   <xacro:property name="motor_constant" value="8.54858e-06" /> <!-- [kg.m/s^2] -->  <!-- still to be determined -->
   <xacro:property name="moment_constant" value="0.016" /> <!-- [m] --> <!-- still to be determined -->
   <xacro:property name="time_constant_up" value="0.0125" /> <!-- [s] --> <!-- still to be determined -->
   <xacro:property name="time_constant_down" value="0.025" /> <!-- [s] --> <!-- still to be determined -->
-  <xacro:property name="max_rot_velocity" value="838" /> <!-- [rad/s] --> <!-- still to be determined -->
+  <xacro:property name="max_rot_velocity_thrust" value="2000" /> <!-- [rad/s] --> <!-- still to be determined -->
+  <xacro:property name="max_rot_velocity_direction" value="1500" /> <!-- [rad/s] --> <!-- still to be determined -->
   <xacro:property name="rotor_drag_coefficient" value="8.06428e-05" /> <!-- still to be determined -->
   <xacro:property name="rolling_moment_coefficient" value="0.000001" /> <!-- still to be determined -->
@@ -37,8 +40,8 @@
   <!-- inertia of a single rotor, assuming it is a cuboid. Height=3mm, width=15mm -->
   <xacro:property name="rotor_inertia_thrust"> <!-- still to be determined -->
-    <xacro:box_inertia x="${radius_rotor_thrust}" y="0.015" z="0.003" mass="${mass_rotor_thrust*rotor_velocity_slowdown_thrust}" />
+    <xacro:box_inertia x="${radius_rotor_thrust_meter}" y="0.015" z="0.003" mass="${mass_rotor_thrust*rotor_velocity_slowdown_thrust}" />
   </xacro:property>
   <xacro:property name="rotor_inertia_direction"> <!-- still to be determined -->
-    <xacro:box_inertia x="${radius_rotor_direction}" y="0.015" z="0.003" mass="${mass_rotor_direction*rotor_velocity_slowdown_direction}" />
+    <xacro:box_inertia x="${radius_rotor_direction_meter}" y="0.015" z="0.003" mass="${mass_rotor_direction*rotor_velocity_slowdown_direction}" />
   </xacro:property>
   <!-- Included URDF Files -->
@@ -64,8 +67,8 @@
     parent="${namespace}/base_link"
     mass_rotor="${mass_rotor_thrust}"
-    radius_rotor="${radius_rotor_thrust}"
-    time_constant_up="${time_constant_up}"
-    time_constant_down="${time_constant_down}"
-    max_rot_velocity="${max_rot_velocity}"
+    radius_rotor="${radius_rotor_thrust_simulation}"
+    time_constant_up="${time_constant_up}"
+    time_constant_down="${time_constant_down}"
+    max_rot_velocity="${max_rot_velocity_thrust}"
     motor_number="2"
     rotor_drag_coefficient="${rotor_drag_coefficient}"
@@ -85,8 +88,8 @@
     parent="${namespace}/base_link"
     mass_rotor="${mass_rotor_thrust}"
-    radius_rotor="${radius_rotor_thrust}"
-    time_constant_up="${time_constant_up}"
-    time_constant_down="${time_constant_down}"
-    max_rot_velocity="${max_rot_velocity}"
+    radius_rotor="${radius_rotor_thrust_simulation}"
+    time_constant_up="${time_constant_up}"
+    time_constant_down="${time_constant_down}"
+    max_rot_velocity="${max_rot_velocity_thrust}"
     motor_number="0"
     rotor_drag_coefficient="${rotor_drag_coefficient}"
@@ -105,8 +108,8 @@
     parent="${namespace}/base_link"
     mass_rotor="${mass_rotor_thrust}"
-    radius_rotor="${radius_rotor_thrust}"
-    time_constant_up="${time_constant_up}"
-    time_constant_down="${time_constant_down}"
-    max_rot_velocity="${max_rot_velocity}"
+    radius_rotor="${radius_rotor_thrust_simulation}"
+    time_constant_up="${time_constant_up}"
+    time_constant_down="${time_constant_down}"
+    max_rot_velocity="${max_rot_velocity_thrust}"
     motor_number="1"
     rotor_drag_coefficient="${rotor_drag_coefficient}"
@@ -125,8 +128,8 @@
     parent="${namespace}/base_link"
     mass_rotor="${mass_rotor_thrust}"
-    radius_rotor="${radius_rotor_thrust}"
-    time_constant_up="${time_constant_up}"
-    time_constant_down="${time_constant_down}"
-    max_rot_velocity="${max_rot_velocity}"
+    radius_rotor="${radius_rotor_thrust_simulation}"
+    time_constant_up="${time_constant_up}"
+    time_constant_down="${time_constant_down}"
+    max_rot_velocity="${max_rot_velocity_thrust}"
     motor_number="3"
     rotor_drag_coefficient="${rotor_drag_coefficient}"
@@ -145,8 +148,8 @@
     parent="${namespace}/base_link"
     mass_rotor="${mass_rotor_direction}"
-    radius_rotor="${radius_rotor_direction}"
-    time_constant_up="${time_constant_up}"
-    time_constant_down="${time_constant_down}"
-    max_rot_velocity="${max_rot_velocity}"
+    radius_rotor="${radius_rotor_direction_simulation}"
+    time_constant_up="${time_constant_up}"
+    time_constant_down="${time_constant_down}"
+    max_rot_velocity="${max_rot_velocity_direction}"
     motor_number="6"
     rotor_drag_coefficient="${rotor_drag_coefficient}"
@@ -165,8 +168,8 @@
     parent="${namespace}/base_link"
     mass_rotor="${mass_rotor_direction}"
-    radius_rotor="${radius_rotor_direction}"
-    time_constant_up="${time_constant_up}"
-    time_constant_down="${time_constant_down}"
-    max_rot_velocity="${max_rot_velocity}"
+    radius_rotor="${radius_rotor_direction_simulation}"
+    time_constant_up="${time_constant_up}"
+    time_constant_down="${time_constant_down}"
+    max_rot_velocity="${max_rot_velocity_direction}"
     motor_number="4"
     rotor_drag_coefficient="${rotor_drag_coefficient}"
@@ -185,8 +188,8 @@
     parent="${namespace}/base_link"
     mass_rotor="${mass_rotor_direction}"
-    radius_rotor="${radius_rotor_direction}"
-    time_constant_up="${time_constant_up}"
-    time_constant_down="${time_constant_down}"
-    max_rot_velocity="${max_rot_velocity}"
+    radius_rotor="${radius_rotor_direction_simulation}"
+    time_constant_up="${time_constant_up}"
+    time_constant_down="${time_constant_down}"
+    max_rot_velocity="${max_rot_velocity_direction}"
     motor_number="5"
     rotor_drag_coefficient="${rotor_drag_coefficient}"
@@ -205,8 +208,8 @@
     parent="${namespace}/base_link"
     mass_rotor="${mass_rotor_direction}"
-    radius_rotor="${radius_rotor_direction}"
-    time_constant_up="${time_constant_up}"
-    time_constant_down="${time_constant_down}"
-    max_rot_velocity="${max_rot_velocity}"
+    radius_rotor="${radius_rotor_direction_simulation}"
+    time_constant_up="${time_constant_up}"
+    time_constant_down="${time_constant_down}"
+    max_rot_velocity="${max_rot_velocity_direction}"
     motor_number="7"
     rotor_drag_coefficient="${rotor_drag_coefficient}"
@@ -219,3 +222,2 @@
   </xacro:vertical_rotor>
 </robot>
-<!-- add channel from omav.xacro-->

Commit message: new rotors

File: rotors_description/urdf/geranos.xacro (robot description, xacro)
@@ -7,8 +7,8 @@
   <xacro:property name="rotor_velocity_slowdown_sim" value="10" />
   <xacro:property name="use_mesh_file" value="true" />
-  <xacro:property name="mesh_file" value="package://rotors_description/meshes/geranos_simple.dae" />
+  <xacro:property name="mesh_file" value="package://rotors_description/meshes/geranos_finalprototyp1.dae" />
   <xacro:property name="mass" value="5.0" /> <!-- [kg] --> <!-- still to be determined -->
   <xacro:property name="body_width" value="0.820" /> <!-- [m] -->
-   <xacro:property name="big_rotor_x" value="0.44017" /> <!-- [m] -->
+   <xacro:property name="big_rotor_x" value="0.440" /> <!-- [m] -->
   <xacro:property name="big_rotor_y" value="0.4098" /> <!-- [m] -->
   <xacro:property name="small_rotor_x" value="0.46506" /> <!-- [m] -->
@@ -22,5 +22,5 @@
   <xacro:property name="rotor_offset_thrust" value="0.13" /> <!-- [m] --> <!-- still to be determined -->
   <xacro:property name="rotor_offset_direction" value="0.27" /> <!-- [m] --> <!-- still to be determined -->
-  <xacro:property name="radius_rotor_thrust_simulation" value="1" /> <!-- [m] --> <!-- radius or durchmesser -->
+  <xacro:property name="radius_rotor_thrust_simulation" value="0.2286" /> <!-- [m] --> <!-- radius or durchmesser -->
   <xacro:property name="radius_rotor_direction_simulation" value="1" /> <!-- [m] --> <!-- radius or durchmesser -->
   <xacro:property name="radius_rotor_thrust_meter" value="0.2286" /> <!-- [m] --> <!-- radius -->
@@ -59,8 +59,8 @@
   </xacro:multirotor_base_macro>
   <!-- Instantiate rotors -->
-  <xacro:vertical_rotor
+  <xacro:thrust_rotor
     robot_namespace="${namespace}"
     suffix="front_right"
-    direction="thrust"
+    direction="propeller_ccw"
     motor_constant="${motor_constant}"
     moment_constant="${moment_constant}"
@@ -79,9 +79,9 @@
     <origin xyz="${big_rotor_x} ${big_rotor_y} ${rotor_offset_thrust}" rpy="0 0 0" />
     <xacro:insert_block name="rotor_inertia_thrust" />
-  </xacro:vertical_rotor>
-  <xacro:vertical_rotor
+  </xacro:thrust_rotor>
+  <xacro:thrust_rotor
     robot_namespace="${namespace}"
     suffix="back_left"
-    direction="thrust"
+    direction="propeller_ccw"
     motor_constant="${motor_constant}"
     moment_constant="${moment_constant}"
@@ -100,8 +100,8 @@
     <origin xyz="-${big_rotor_x} -${big_rotor_y} ${rotor_offset_thrust}" rpy="0 0 0" />
     <xacro:insert_block name="rotor_inertia_thrust" />
-  </xacro:vertical_rotor>
-  <xacro:vertical_rotor robot_namespace="${namespace}"
+  </xacro:thrust_rotor>
+  <xacro:thrust_rotor robot_namespace="${namespace}"
     suffix="back_right"
-    direction="thrust"
+    direction="propeller_cw"
     motor_constant="${motor_constant}"
     moment_constant="${moment_constant}"
@@ -120,8 +120,8 @@
     <origin xyz="-${big_rotor_x} ${big_rotor_y} ${rotor_offset_thrust}" rpy="0 0 0" />
     <xacro:insert_block name="rotor_inertia_thrust" />
-  </xacro:vertical_rotor>
-  <xacro:vertical_rotor robot_namespace="${namespace}"
+  </xacro:thrust_rotor>
+  <xacro:thrust_rotor robot_namespace="${namespace}"
     suffix="front_left"
-    direction="thrust"
+    direction="propeller_cw"
     motor_constant="${motor_constant}"
     moment_constant="${moment_constant}"
@@ -140,8 +140,8 @@
     <origin xyz="${big_rotor_x} -${big_rotor_y} ${rotor_offset_thrust}" rpy="0 0 0" />
     <xacro:insert_block name="rotor_inertia_thrust" />
-  </xacro:vertical_rotor>
-<xacro:vertical_rotor robot_namespace="${namespace}"
+  </xacro:thrust_rotor>
+<xacro:direction_rotor robot_namespace="${namespace}"
     suffix="direction_front"
-    direction="direction"
+    direction="direction_cw"
     motor_constant="${motor_constant}"
     moment_constant="${moment_constant}"
@@ -158,10 +158,10 @@
     use_own_mesh="false"
     mesh="">
-    <origin xyz="${small_rotor_x}  0 ${rotor_offset_direction}" rpy="0 -0.698132 0" />
-    <xacro:insert_block name="rotor_inertia_direction" />
-  </xacro:vertical_rotor>
-  <xacro:vertical_rotor robot_namespace="${namespace}"
+    <origin xyz="${small_rotor_x}  0 ${rotor_offset_direction}" rpy="0 -0.837758 0" />
+    <xacro:insert_block name="rotor_inertia_direction" />
+  </xacro:direction_rotor>
+  <xacro:direction_rotor robot_namespace="${namespace}"
     suffix="direciton_back"
-    direction="direction"
+    direction="direction_cw"
     motor_constant="${motor_constant}"
     moment_constant="${moment_constant}"
@@ -178,10 +178,10 @@
     use_own_mesh="false"
     mesh="">
-    <origin xyz="-${small_rotor_x} 0 ${rotor_offset_direction}" rpy="0 0.698132 0" />
-    <xacro:insert_block name="rotor_inertia_direction" />
-  </xacro:vertical_rotor>
-  <xacro:vertical_rotor robot_namespace="${namespace}"
+    <origin xyz="-${small_rotor_x} 0 ${rotor_offset_direction}" rpy="0 0.837758 0" />
+    <xacro:insert_block name="rotor_inertia_direction" />
+  </xacro:direction_rotor>
+  <xacro:direction_rotor robot_namespace="${namespace}"
     suffix="direction_right"
-    direction="direction"
+    direction="direction_ccw"
     motor_constant="${motor_constant}"
     moment_constant="${moment_constant}"
@@ -198,10 +198,10 @@
     use_own_mesh="false"
     mesh="">
-    <origin xyz="0 ${small_rotor_y}  ${rotor_offset_direction}" rpy="0.698132 0 0" />
-    <xacro:insert_block name="rotor_inertia_direction" />
-  </xacro:vertical_rotor>
-  <xacro:vertical_rotor robot_namespace="${namespace}"
+    <origin xyz="0 ${small_rotor_y}  ${rotor_offset_direction}" rpy="0.837758 0 0" />
+    <xacro:insert_block name="rotor_inertia_direction" />
+  </xacro:direction_rotor>
+  <xacro:direction_rotor robot_namespace="${namespace}"
     suffix="direction_left"
-    direction="direction"
+    direction="direction_ccw"
     motor_constant="${motor_constant}"
     moment_constant="${moment_constant}"
@@ -218,6 +218,6 @@
     use_own_mesh="false"
     mesh="">
-    <origin xyz="0 -${small_rotor_y}  ${rotor_offset_direction}" rpy="-0.698132 0 0" />
-    <xacro:insert_block name="rotor_inertia_direction" />
-  </xacro:vertical_rotor>
+    <origin xyz="0 -${small_rotor_y}  ${rotor_offset_direction}" rpy="-0.837758 0 0" />
+    <xacro:insert_block name="rotor_inertia_direction" />
+  </xacro:direction_rotor>
 </robot>

File: rotors_description/urdf/multirotor_base.xacro (robot description, xacro)
@@ -35,4 +35,5 @@
     params="robot_namespace mass body_width body_height use_mesh_file mesh_file *inertia">
     <link name="${robot_namespace}/base_link"></link>
+    <!-- origin -->
     <joint name="${robot_namespace}/base_joint" type="fixed">
       <origin xyz="0 0 0" rpy="0 0 0" />
@@ -73,10 +74,10 @@
     </gazebo>
   </xacro:macro>
-  <!-- Rotor joint and link -->
-  <xacro:macro name="vertical_rotor"
+  <!-- Thrust Rotor joint and link -->
+  <xacro:macro name="thrust_rotor"
     params="robot_namespace suffix direction motor_constant moment_constant parent mass_rotor radius_rotor time_constant_up time_constant_down max_rot_velocity motor_number rotor_drag_coefficient rolling_moment_coefficient color use_own_mesh mesh *origin *inertia">
     <joint name="${robot_namespace}/rotor_${motor_number}_joint" type="continuous">
       <xacro:insert_block name="origin" />
-      <axis xyz="0 0 1" />
+      <axis xyz="0 0 1" rpy="0 0 0"/>
       <!-- TODO(ff): not currently set because it's not yet supported -->
       <!-- <limit effort="2000" velocity="${max_rot_velocity}" /> -->
@@ -132,3 +133,62 @@
     </gazebo>
   </xacro:macro>
+  <!-- Direction Rotor joint and link -->
+  <xacro:macro name="direction_rotor"
+    params="robot_namespace suffix direction motor_constant moment_constant parent mass_rotor radius_rotor time_constant_up time_constant_down max_rot_velocity motor_number rotor_drag_coefficient rolling_moment_coefficient color use_own_mesh mesh *origin *inertia">
+    <joint name="${robot_namespace}/rotor_${motor_number}_joint" type="continuous">
+      <xacro:insert_block name="origin" />
+      <axis xyz="0 0 1" rpy="0 0 0"/>
+      <!-- TODO(ff): not currently set because it's not yet supported -->
+      <!-- <limit effort="2000" velocity="${max_rot_velocity}" /> -->
+      <parent link="${parent}" />
+      <child link="${robot_namespace}/rotor_${motor_number}" />
+    </joint>
+    <link name="${robot_namespace}/rotor_${motor_number}">
+      <inertial>
+        <mass value="${mass_rotor_direction}" /> <!-- [kg] -->
+        <xacro:insert_block name="inertia" />
+      </inertial>
+      <visual>
+        <geometry>
+          <!-- <cylinder length="0.005" radius="${radius_rotor}"/> --> <!-- [m] -->
+          <xacro:if value="${use_own_mesh}">
+            <mesh filename="${mesh}"
+              scale="1 1 1" />
+          </xacro:if>
+          <xacro:unless value="${use_own_mesh}">
+            <mesh filename="package://rotors_description/meshes/geranos_prop_${direction}.dae"
+              scale="${radius_rotor} ${radius_rotor} ${radius_rotor}" /> <!-- The propeller meshes have a radius of 1m -->
+            <!-- <box size="${2*radius_rotor} 0.01 0.005"/> -->
+          </xacro:unless>
+        </geometry>
+      </visual>
+      <collision>
+        <geometry>
+          <cylinder length="0.005" radius="${radius_rotor}" /> <!-- [m] -->
+        </geometry>
+      </collision>
+    </link>
+    <gazebo>
+      <plugin name="${robot_namespace}_${suffix}_motor_model" filename="librotors_gazebo_motor_model.so">
+        <robotNamespace>${robot_namespace}</robotNamespace>
+        <jointName>${robot_namespace}/rotor_${motor_number}_joint</jointName>
+        <linkName>${robot_namespace}/rotor_${motor_number}</linkName>
+        <turningDirection>${direction}</turningDirection>
+        <timeConstantUp>${time_constant_up}</timeConstantUp>
+        <timeConstantDown>${time_constant_down}</timeConstantDown>
+        <maxRotVelocity>${max_rot_velocity}</maxRotVelocity>
+        <motorConstant>${motor_constant}</motorConstant>
+        <momentConstant>${moment_constant}</momentConstant>
+        <commandSubTopic>gazebo/command/motor_speed</commandSubTopic>
+        <motorNumber>${motor_number}</motorNumber>
+        <rotorDragCoefficient>${rotor_drag_coefficient}</rotorDragCoefficient>
+        <rollingMomentCoefficient>${rolling_moment_coefficient}</rollingMomentCoefficient>
+        <motorSpeedPubTopic>motor_speed/${motor_number}</motorSpeedPubTopic>
+        <rotorVelocitySlowdownSim>${rotor_velocity_slowdown_direction}</rotorVelocitySlowdownSim>
+      </plugin>
+    </gazebo>
+    <gazebo reference="${robot_namespace}/rotor_${motor_number}">
+      <material>Gazebo/${color}</material>
+    </gazebo>
+  </xacro:macro>
 </robot>

Commit message: changes to cw ccw direction

File: rotors_description/urdf/geranos.xacro (robot description, xacro)
@@ -62,5 +62,5 @@
     robot_namespace="${namespace}"
     suffix="front_right"
-    direction="propeller_ccw"
+    direction="ccw"
     motor_constant="${motor_constant}"
     moment_constant="${moment_constant}"
@@ -83,5 +83,5 @@
     robot_namespace="${namespace}"
     suffix="back_left"
-    direction="propeller_ccw"
+    direction="ccw"
     motor_constant="${motor_constant}"
     moment_constant="${moment_constant}"
@@ -103,5 +103,5 @@
   <xacro:thrust_rotor robot_namespace="${namespace}"
     suffix="back_right"
-    direction="propeller_cw"
+    direction="cw"
     motor_constant="${motor_constant}"
     moment_constant="${moment_constant}"
@@ -123,5 +123,5 @@
   <xacro:thrust_rotor robot_namespace="${namespace}"
     suffix="front_left"
-    direction="propeller_cw"
+    direction="cw"
     motor_constant="${motor_constant}"
     moment_constant="${moment_constant}"
@@ -143,5 +143,5 @@
 <xacro:direction_rotor robot_namespace="${namespace}"
     suffix="direction_front"
-    direction="direction_cw"
+    direction="cw"
     motor_constant="${motor_constant}"
     moment_constant="${moment_constant}"
@@ -163,5 +163,5 @@
   <xacro:direction_rotor robot_namespace="${namespace}"
     suffix="direciton_back"
-    direction="direction_cw"
+    direction="cw"
     motor_constant="${motor_constant}"
     moment_constant="${moment_constant}"
@@ -183,5 +183,5 @@
   <xacro:direction_rotor robot_namespace="${namespace}"
     suffix="direction_right"
-    direction="direction_ccw"
+    direction="ccw"
     motor_constant="${motor_constant}"
     moment_constant="${moment_constant}"
@@ -203,5 +203,5 @@
   <xacro:direction_rotor robot_namespace="${namespace}"
     suffix="direction_left"
-    direction="direction_ccw"
+    direction="ccw"
     motor_constant="${motor_constant}"
     moment_constant="${moment_constant}"

File: rotors_description/urdf/multirotor_base.xacro (robot description, xacro)
@@ -157,5 +157,5 @@
           </xacro:if>
           <xacro:unless value="${use_own_mesh}">
-            <mesh filename="package://rotors_description/meshes/geranos_prop_${direction}.dae"
+            <mesh filename="package://rotors_description/meshes/geranos_direction_${direction}.dae"
               scale="${radius_rotor} ${radius_rotor} ${radius_rotor}" /> <!-- The propeller meshes have a radius of 1m -->
             <!-- <box size="${2*radius_rotor} 0.01 0.005"/> -->

Commit message: adjusting parameters to yaml file

File: rotors_description/urdf/geranos.xacro (robot description, xacro)
@@ -10,8 +10,8 @@
   <xacro:property name="mass" value="5.0" /> <!-- [kg] --> <!-- still to be determined -->
   <xacro:property name="body_width" value="0.820" /> <!-- [m] -->
-   <xacro:property name="big_rotor_x" value="0.440" /> <!-- [m] -->
+   <xacro:property name="big_rotor_x" value="0.44017" /> <!-- [m] -->
   <xacro:property name="big_rotor_y" value="0.4098" /> <!-- [m] -->
-  <xacro:property name="small_rotor_x" value="0.46506" /> <!-- [m] -->
-  <xacro:property name="small_rotor_y" value="0.36506" /> <!-- [m] -->
+  <xacro:property name="small_rotor_x" value="0.4481" /> <!-- [m] -->
+  <xacro:property name="small_rotor_y" value="0.3481" /> <!-- [m] -->
   <xacro:property name="half_body_width" value="0.3" /> <!-- [m] -->
   <xacro:property name="side_length_one" value="0.2" /> <!-- [m] -->
@@ -143,5 +143,5 @@
 <xacro:direction_rotor robot_namespace="${namespace}"
     suffix="direction_front"
-    direction="cw"
+    direction="ccw"
     motor_constant="${motor_constant}"
     moment_constant="${moment_constant}"
@@ -203,5 +203,5 @@
   <xacro:direction_rotor robot_namespace="${namespace}"
     suffix="direction_left"
-    direction="ccw"
+    direction="cw"
     motor_constant="${motor_constant}"
     moment_constant="${moment_constant}"
