Commit message: Improvement of the blue rotors and visual dae-rotor-files

File: rotors_description/urdf/geranos.xacro (robot description, xacro)
@@ -10,8 +10,9 @@
   <xacro:property name="mass" value="5.0" /> <!-- [kg] --> <!-- still to be determined -->
   <xacro:property name="body_width" value="0.820" /> <!-- [m] -->
-   <xacro:property name="big_rotor_x" value="0.44017" /> <!-- [m] -->
+  <xacro:property name="big_rotor_x" value="0.44017" /> <!-- [m] -->
   <xacro:property name="big_rotor_y" value="0.4098" /> <!-- [m] -->
-  <xacro:property name="small_rotor_x" value="0.4481" /> <!-- [m] -->
-  <xacro:property name="small_rotor_y" value="0.3481" /> <!-- [m] -->
+  <xacro:property name="small_rotor_x" value="0.463" /> <!-- [m] -->
+  <xacro:property name="small_rotor_y" value="0.363" /> <!-- [m] -->
+  <xacro:property name="small_rotor_x_off" value="0.4547" /> <!-- [m] -->
   <xacro:property name="half_body_width" value="0.3" /> <!-- [m] -->
   <xacro:property name="side_length_one" value="0.2" /> <!-- [m] -->
@@ -21,6 +22,7 @@
   <xacro:property name="mass_rotor_direction" value="0.005" /> <!-- [kg] --> <!-- still to be determined -->
   <xacro:property name="rotor_offset_thrust" value="0.13" /> <!-- [m] --> <!-- still to be determined -->
-  <xacro:property name="rotor_offset_direction" value="0.27" /> <!-- [m] --> <!-- still to be determined -->
-  <xacro:property name="radius_rotor_thrust_simulation" value="0.2286" /> <!-- [m] --> <!-- radius or durchmesser -->
+  <xacro:property name="rotor_offset_direction" value="0.267" /> <!-- [m] --> <!-- still to be determined -->
+  <xacro:property name="rotor_offset_direction_off" value="0.274" /> <!-- [m] --> <!-- still to be determined -->
+  <xacro:property name="radius_rotor_thrust_simulation" value="1" /> <!-- [m] --> <!-- radius or durchmesser -->
   <xacro:property name="radius_rotor_direction_simulation" value="1" /> <!-- [m] --> <!-- radius or durchmesser -->
   <xacro:property name="radius_rotor_thrust_meter" value="0.2286" /> <!-- [m] --> <!-- radius -->
@@ -74,5 +76,5 @@
     rotor_drag_coefficient="${rotor_drag_coefficient}"
     rolling_moment_coefficient="${rolling_moment_coefficient}"
-    color="Red"
+    color="Yellow"
     use_own_mesh="false"
     mesh="">
@@ -141,7 +143,7 @@
     <xacro:insert_block name="rotor_inertia_thrust" />
   </xacro:thrust_rotor>
-<xacro:direction_rotor robot_namespace="${namespace}"
+<xacro:direction_f_rotor robot_namespace="${namespace}"
     suffix="direction_front"
-    direction="ccw"
+    direction="cw"
     motor_constant="${motor_constant}"
     moment_constant="${moment_constant}"
@@ -160,6 +162,6 @@
     <origin xyz="${small_rotor_x}  0 ${rotor_offset_direction}" rpy="0 -0.837758 0" />
     <xacro:insert_block name="rotor_inertia_direction" />
-  </xacro:direction_rotor>
-  <xacro:direction_rotor robot_namespace="${namespace}"
+  </xacro:direction_f_rotor>
+  <xacro:direction_b_rotor robot_namespace="${namespace}"
     suffix="direciton_back"
     direction="cw"
@@ -178,8 +180,8 @@
     use_own_mesh="false"
     mesh="">
-    <origin xyz="-${small_rotor_x} 0 ${rotor_offset_direction}" rpy="0 0.837758 0" />
-    <xacro:insert_block name="rotor_inertia_direction" />
-  </xacro:direction_rotor>
-  <xacro:direction_rotor robot_namespace="${namespace}"
+    <origin xyz="-${small_rotor_x_off} 0 ${rotor_offset_direction_off}" rpy="0 0.837758 0" />
+    <xacro:insert_block name="rotor_inertia_direction" />
+  </xacro:direction_b_rotor>
+  <xacro:direction_r_rotor robot_namespace="${namespace}"
     suffix="direction_right"
     direction="ccw"
@@ -200,8 +202,8 @@
     <origin xyz="0 ${small_rotor_y}  ${rotor_offset_direction}" rpy="0.837758 0 0" />
     <xacro:insert_block name="rotor_inertia_direction" />
-  </xacro:direction_rotor>
-  <xacro:direction_rotor robot_namespace="${namespace}"
+  </xacro:direction_r_rotor>
+  <xacro:direction_l_rotor robot_namespace="${namespace}"
     suffix="direction_left"
-    direction="cw"
+    direction="ccw"
     motor_constant="${motor_constant}"
     moment_constant="${moment_constant}"
@@ -220,4 +222,4 @@
     <origin xyz="0 -${small_rotor_y}  ${rotor_offset_direction}" rpy="-0.837758 0 0" />
     <xacro:insert_block name="rotor_inertia_direction" />
-  </xacro:direction_rotor>
+  </xacro:direction_l_rotor>
 </robot>

File: rotors_description/urdf/multirotor_base.xacro (robot description, xacro)
@@ -37,5 +37,5 @@
     <!-- origin -->
     <joint name="${robot_namespace}/base_joint" type="fixed">
-      <origin xyz="0 0 0" rpy="0 0 0" />
+      <origin xyz="0.001 0 0" rpy="0 0 0" />
       <parent link="${robot_namespace}/base_link" />
       <child link="${robot_namespace}/base_link_inertia" />
@@ -48,5 +48,5 @@
       </inertial>
       <visual>
-        <origin xyz="0 0 0" rpy="0 0 0" />
+        <origin xyz="0.001 0 0" rpy="0 0 0" />
         <geometry>
           <xacro:if value="${use_mesh_file}">
@@ -88,5 +88,5 @@
       <inertial>
         <mass value="${mass_rotor_thrust}" /> <!-- [kg] -->
-        <xacro:insert_block name="inertia" />
+        <xacro:insert_block name="rotor_inertia_thrust" />
       </inertial>
       <visual>
@@ -106,5 +106,5 @@
       <collision>
         <geometry>
-          <cylinder length="0.005" radius="${radius_rotor}" /> <!-- [m] -->
+          <cylinder length="0.007" radius="${radius_rotor}" /> <!-- [m] -->
         </geometry>
       </collision>
@@ -134,9 +134,10 @@
   </xacro:macro>
   <!-- Direction Rotor joint and link -->
-  <xacro:macro name="direction_rotor"
-    params="robot_namespace suffix direction motor_constant moment_constant parent mass_rotor radius_rotor time_constant_up time_constant_down max_rot_velocity motor_number rotor_drag_coefficient rolling_moment_coefficient color use_own_mesh mesh *origin *inertia">
-    <joint name="${robot_namespace}/rotor_${motor_number}_joint" type="continuous">
-      <xacro:insert_block name="origin" />
-      <axis xyz="0 0 1" rpy="0 0 0"/>
+  <xacro:macro name="direction_f_rotor"
+    params="robot_namespace suffix direction motor_constant moment_constant parent mass_rotor radius_rotor time_constant_up time_constant_down max_rot_velocity motor_number rotor_drag_coefficient rolling_moment_coefficient color use_own_mesh mesh *origin *inertia">
+    <joint name="${robot_namespace}/rotor_${motor_number}_joint" type="continuous">
+      <xacro:insert_block name="origin" />
+      <axis xyz="0 0 1" rpy="0 -0.837758 0"/>
+      <origin xyz="0.463 0 0.267" rpy="0 0 0" />
       <!-- TODO(ff): not currently set because it's not yet supported -->
       <!-- <limit effort="2000" velocity="${max_rot_velocity}" /> -->
@@ -147,5 +148,5 @@
       <inertial>
         <mass value="${mass_rotor_direction}" /> <!-- [kg] -->
-        <xacro:insert_block name="inertia" />
+        <xacro:insert_block name="rotor_inertia_direction" />
       </inertial>
       <visual>
@@ -165,5 +166,5 @@
       <collision>
         <geometry>
-          <cylinder length="0.005" radius="${radius_rotor}" /> <!-- [m] -->
+          <cylinder length="0.007" radius="${radius_rotor}" /> <!-- [m] -->
         </geometry>
       </collision>
@@ -192,3 +193,183 @@
     </gazebo>
   </xacro:macro>
+<!-- Direction Rotor joint and link -->
+  <xacro:macro name="direction_b_rotor"
+    params="robot_namespace suffix direction motor_constant moment_constant parent mass_rotor radius_rotor time_constant_up time_constant_down max_rot_velocity motor_number rotor_drag_coefficient rolling_moment_coefficient color use_own_mesh mesh *origin *inertia">
+    <joint name="${robot_namespace}/rotor_${motor_number}_joint" type="continuous">
+      <xacro:insert_block name="origin" />
+      <axis xyz="0 0 1" rpy="0 0.837758 0"/>
+      <origin xyz="-0.4547 0 0.274" rpy="0 0 0" />
+      <!-- TODO(ff): not currently set because it's not yet supported -->
+      <!-- <limit effort="2000" velocity="${max_rot_velocity}" /> -->
+      <parent link="${parent}" />
+      <child link="${robot_namespace}/rotor_${motor_number}" />
+    </joint>
+    <link name="${robot_namespace}/rotor_${motor_number}">
+      <inertial>
+        <mass value="${mass_rotor_direction}" /> <!-- [kg] -->
+        <xacro:insert_block name="rotor_inertia_direction" />
+      </inertial>
+      <visual>
+        <geometry>
+          <!-- <cylinder length="0.005" radius="${radius_rotor}"/> --> <!-- [m] -->
+          <xacro:if value="${use_own_mesh}">
+            <mesh filename="${mesh}"
+              scale="1 1 1" />
+          </xacro:if>
+          <xacro:unless value="${use_own_mesh}">
+            <mesh filename="package://rotors_description/meshes/geranos_direction_${direction}.dae"
+              scale="${radius_rotor} ${radius_rotor} ${radius_rotor}" /> <!-- The propeller meshes have a radius of 1m -->
+            <!-- <box size="${2*radius_rotor} 0.01 0.005"/> -->
+          </xacro:unless>
+        </geometry>
+      </visual>
+      <collision>
+        <geometry>
+          <cylinder length="0.007" radius="${radius_rotor}" /> <!-- [m] -->
+        </geometry>
+      </collision>
+    </link>
+    <gazebo>
+      <plugin name="${robot_namespace}_${suffix}_motor_model" filename="librotors_gazebo_motor_model.so">
+        <robotNamespace>${robot_namespace}</robotNamespace>
+        <jointName>${robot_namespace}/rotor_${motor_number}_joint</jointName>
+        <linkName>${robot_namespace}/rotor_${motor_number}</linkName>
+        <turningDirection>${direction}</turningDirection>
+        <timeConstantUp>${time_constant_up}</timeConstantUp>
+        <timeConstantDown>${time_constant_down}</timeConstantDown>
+        <maxRotVelocity>${max_rot_velocity}</maxRotVelocity>
+        <motorConstant>${motor_constant}</motorConstant>
+        <momentConstant>${moment_constant}</momentConstant>
+        <commandSubTopic>gazebo/command/motor_speed</commandSubTopic>
+        <motorNumber>${motor_number}</motorNumber>
+        <rotorDragCoefficient>${rotor_drag_coefficient}</rotorDragCoefficient>
+        <rollingMomentCoefficient>${rolling_moment_coefficient}</rollingMomentCoefficient>
+        <motorSpeedPubTopic>motor_speed/${motor_number}</motorSpeedPubTopic>
+        <rotorVelocitySlowdownSim>${rotor_velocity_slowdown_direction}</rotorVelocitySlowdownSim>
+      </plugin>
+    </gazebo>
+    <gazebo reference="${robot_namespace}/rotor_${motor_number}">
+      <material>Gazebo/${color}</material>
+    </gazebo>
+  </xacro:macro>
+<!-- Direction Rotor joint and link -->
+  <xacro:macro name="direction_r_rotor"
+    params="robot_namespace suffix direction motor_constant moment_constant parent mass_rotor radius_rotor time_constant_up time_constant_down max_rot_velocity motor_number rotor_drag_coefficient rolling_moment_coefficient color use_own_mesh mesh *origin *inertia">
+    <joint name="${robot_namespace}/rotor_${motor_number}_joint" type="continuous">
+      <xacro:insert_block name="origin" />
+      <axis xyz="0 0 1" rpy="0.837758 0 0"/>
+      <origin xyz="0 0.363 0.267" rpy="0 0 0" />
+      <!-- TODO(ff): not currently set because it's not yet supported -->
+      <!-- <limit effort="2000" velocity="${max_rot_velocity}" /> -->
+      <parent link="${parent}" />
+      <child link="${robot_namespace}/rotor_${motor_number}" />
+    </joint>
+    <link name="${robot_namespace}/rotor_${motor_number}">
+      <inertial>
+        <mass value="${mass_rotor_direction}" /> <!-- [kg] -->
+        <xacro:insert_block name="rotor_inertia_direction" />
+      </inertial>
+      <visual>
+        <geometry>
+          <!-- <cylinder length="0.005" radius="${radius_rotor}"/> --> <!-- [m] -->
+          <xacro:if value="${use_own_mesh}">
+            <mesh filename="${mesh}"
+              scale="1 1 1" />
+          </xacro:if>
+          <xacro:unless value="${use_own_mesh}">
+            <mesh filename="package://rotors_description/meshes/geranos_direction_${direction}.dae"
+              scale="${radius_rotor} ${radius_rotor} ${radius_rotor}" /> <!-- The propeller meshes have a radius of 1m -->
+            <!-- <box size="${2*radius_rotor} 0.01 0.005"/> -->
+          </xacro:unless>
+        </geometry>
+      </visual>
+      <collision>
+        <geometry>
+          <cylinder length="0.007" radius="${radius_rotor}" /> <!-- [m] -->
+        </geometry>
+      </collision>
+    </link>
+    <gazebo>
+      <plugin name="${robot_namespace}_${suffix}_motor_model" filename="librotors_gazebo_motor_model.so">
+        <robotNamespace>${robot_namespace}</robotNamespace>
+        <jointName>${robot_namespace}/rotor_${motor_number}_joint</jointName>
+        <linkName>${robot_namespace}/rotor_${motor_number}</linkName>
+        <turningDirection>${direction}</turningDirection>
+        <timeConstantUp>${time_constant_up}</timeConstantUp>
+        <timeConstantDown>${time_constant_down}</timeConstantDown>
+        <maxRotVelocity>${max_rot_velocity}</maxRotVelocity>
+        <motorConstant>${motor_constant}</motorConstant>
+        <momentConstant>${moment_constant}</momentConstant>
+        <commandSubTopic>gazebo/command/motor_speed</commandSubTopic>
+        <motorNumber>${motor_number}</motorNumber>
+        <rotorDragCoefficient>${rotor_drag_coefficient}</rotorDragCoefficient>
+        <rollingMomentCoefficient>${rolling_moment_coefficient}</rollingMomentCoefficient>
+        <motorSpeedPubTopic>motor_speed/${motor_number}</motorSpeedPubTopic>
+        <rotorVelocitySlowdownSim>${rotor_velocity_slowdown_direction}</rotorVelocitySlowdownSim>
+      </plugin>
+    </gazebo>
+    <gazebo reference="${robot_namespace}/rotor_${motor_number}">
+      <material>Gazebo/${color}</material>
+    </gazebo>
+  </xacro:macro>
+<!-- Direction Rotor joint and link -->
+  <xacro:macro name="direction_l_rotor"
+    params="robot_namespace suffix direction motor_constant moment_constant parent mass_rotor radius_rotor time_constant_up time_constant_down max_rot_velocity motor_number rotor_drag_coefficient rolling_moment_coefficient color use_own_mesh mesh *origin *inertia">
+    <joint name="${robot_namespace}/rotor_${motor_number}_joint" type="continuous">
+      <xacro:insert_block name="origin" />
+      <axis xyz="0 0 1" rpy="-0.837758 0 0"/>
+      <origin xyz="0 -0.363 0.267" rpy="0 0 0" />
+      <!-- TODO(ff): not currently set because it's not yet supported -->
+      <!-- <limit effort="2000" velocity="${max_rot_velocity}" /> -->
+      <parent link="${parent}" />
+      <child link="${robot_namespace}/rotor_${motor_number}" />
+    </joint>
+    <link name="${robot_namespace}/rotor_${motor_number}">
+      <inertial>
+        <mass value="${mass_rotor_direction}" /> <!-- [kg] -->
+        <xacro:insert_block name="rotor_inertia_direction" />
+      </inertial>
+      <visual>
+        <geometry>
+          <!-- <cylinder length="0.005" radius="${radius_rotor}"/> --> <!-- [m] -->
+          <xacro:if value="${use_own_mesh}">
+            <mesh filename="${mesh}"
+              scale="1 1 1" />
+          </xacro:if>
+          <xacro:unless value="${use_own_mesh}">
+            <mesh filename="package://rotors_description/meshes/geranos_direction_${direction}.dae"
+              scale="${radius_rotor} ${radius_rotor} ${radius_rotor}" /> <!-- The propeller meshes have a radius of 1m -->
+            <!-- <box size="${2*radius_rotor} 0.01 0.005"/> -->
+          </xacro:unless>
+        </geometry>
+      </visual>
+      <collision>
+        <geometry>
+          <cylinder length="0.007" radius="${radius_rotor}" /> <!-- [m] -->
+        </geometry>
+      </collision>
+    </link>
+    <gazebo>
+      <plugin name="${robot_namespace}_${suffix}_motor_model" filename="librotors_gazebo_motor_model.so">
+        <robotNamespace>${robot_namespace}</robotNamespace>
+        <jointName>${robot_namespace}/rotor_${motor_number}_joint</jointName>
+        <linkName>${robot_namespace}/rotor_${motor_number}</linkName>
+        <turningDirection>${direction}</turningDirection>
+        <timeConstantUp>${time_constant_up}</timeConstantUp>
+        <timeConstantDown>${time_constant_down}</timeConstantDown>
+        <maxRotVelocity>${max_rot_velocity}</maxRotVelocity>
+        <motorConstant>${motor_constant}</motorConstant>
+        <momentConstant>${moment_constant}</momentConstant>
+        <commandSubTopic>gazebo/command/motor_speed</commandSubTopic>
+        <motorNumber>${motor_number}</motorNumber>
+        <rotorDragCoefficient>${rotor_drag_coefficient}</rotorDragCoefficient>
+        <rollingMomentCoefficient>${rolling_moment_coefficient}</rollingMomentCoefficient>
+        <motorSpeedPubTopic>motor_speed/${motor_number}</motorSpeedPubTopic>
+        <rotorVelocitySlowdownSim>${rotor_velocity_slowdown_direction}</rotorVelocitySlowdownSim>
+      </plugin>
+    </gazebo>
+    <gazebo reference="${robot_namespace}/rotor_${motor_number}">
+      <material>Gazebo/${color}</material>
+    </gazebo>
+  </xacro:macro>
 </robot>

File: rotors_gazebo/models/rotors_description/urdf/multirotor_base.xacro (robot description, xacro)
@@ -72,6 +72,6 @@
    </gazebo>
   </xacro:macro>
-  <!-- Rotor joint and link -->
-  <xacro:macro name="vertical_rotor"
+  <!-- Thrust_Rotor joint and link -->
+  <xacro:macro name="thrust_rotor"
     params="robot_namespace suffix direction motor_constant moment_constant parent mass_rotor radius_rotor time_constant_up time_constant_down max_rot_velocity motor_number rotor_drag_coefficient rolling_moment_coefficient color mesh mesh_scale *origin *inertia">
     <joint name="rotor_${motor_number}_joint" type="continuous">
@@ -140,3 +140,62 @@
     </gazebo>
   </xacro:macro>
+  <!-- Direction Rotor joint and link -->
+  <xacro:macro name="direction_rotor"
+    params="robot_namespace suffix direction motor_constant moment_constant parent mass_rotor radius_rotor time_constant_up time_constant_down max_rot_velocity motor_number rotor_drag_coefficient rolling_moment_coefficient color use_own_mesh mesh *origin *inertia">
+    <joint name="${robot_namespace}/rotor_${motor_number}_joint" type="continuous">
+      <xacro:insert_block name="origin" />
+      <axis xyz="0 0 1" rpy="0 0 0"/>
+      <!-- TODO(ff): not currently set because it's not yet supported -->
+      <!-- <limit effort="2000" velocity="${max_rot_velocity}" /> -->
+      <parent link="${parent}" />
+      <child link="${robot_namespace}/rotor_${motor_number}" />
+    </joint>
+    <link name="${robot_namespace}/rotor_${motor_number}">
+      <inertial>
+        <mass value="${mass_rotor_direction}" /> <!-- [kg] -->
+        <xacro:insert_block name="rotor_inertia_direction" />
+      </inertial>
+      <visual>
+        <geometry>
+          <!-- <cylinder length="0.005" radius="${radius_rotor}"/> --> <!-- [m] -->
+          <xacro:if value="${use_own_mesh}">
+            <mesh filename="${mesh}"
+              scale="1 1 1" />
+          </xacro:if>
+          <xacro:unless value="${use_own_mesh}">
+            <mesh filename="package://rotors_description/meshes/geranos_direction_${direction}.dae"
+              scale="${radius_rotor} ${radius_rotor} ${radius_rotor}" /> <!-- The propeller meshes have a radius of 1m -->
+            <!-- <box size="${2*radius_rotor} 0.01 0.005"/> -->
+          </xacro:unless>
+        </geometry>
+      </visual>
+      <collision>
+        <geometry>
+          <cylinder length="0.007" radius="${radius_rotor}" /> <!-- [m] -->
+        </geometry>
+      </collision>
+    </link>
+    <gazebo>
+      <plugin name="${robot_namespace}_${suffix}_motor_model" filename="librotors_gazebo_motor_model.so">
+        <robotNamespace>${robot_namespace}</robotNamespace>
+        <jointName>${robot_namespace}/rotor_${motor_number}_joint</jointName>
+        <linkName>${robot_namespace}/rotor_${motor_number}</linkName>
+        <turningDirection>${direction}</turningDirection>
+        <timeConstantUp>${time_constant_up}</timeConstantUp>
+        <timeConstantDown>${time_constant_down}</timeConstantDown>
+        <maxRotVelocity>${max_rot_velocity}</maxRotVelocity>
+        <motorConstant>${motor_constant}</motorConstant>
+        <momentConstant>${moment_constant}</momentConstant>
+        <commandSubTopic>gazebo/command/motor_speed</commandSubTopic>
+        <motorNumber>${motor_number}</motorNumber>
+        <rotorDragCoefficient>${rotor_drag_coefficient}</rotorDragCoefficient>
+        <rollingMomentCoefficient>${rolling_moment_coefficient}</rollingMomentCoefficient>
+        <motorSpeedPubTopic>motor_speed/${motor_number}</motorSpeedPubTopic>
+        <rotorVelocitySlowdownSim>${rotor_velocity_slowdown_direction}</rotorVelocitySlowdownSim>
+      </plugin>
+    </gazebo>
+    <gazebo reference="${robot_namespace}/rotor_${motor_number}">
+      <material>Gazebo/${color}</material>
+    </gazebo>
+  </xacro:macro>
 </robot>

Commit message: modified max rotor velocities

File: rotors_description/urdf/geranos.xacro (robot description, xacro)
@@ -33,5 +33,5 @@
   <xacro:property name="time_constant_down" value="0.025" /> <!-- [s] --> <!-- still to be determined -->
   <xacro:property name="max_rot_velocity_thrust" value="2000" /> <!-- [rad/s] --> <!-- still to be determined -->
-  <xacro:property name="max_rot_velocity_direction" value="1500" /> <!-- [rad/s] --> <!-- still to be determined -->
+  <xacro:property name="max_rot_velocity_direction" value="2000" /> <!-- [rad/s] --> <!-- still to be determined -->
   <xacro:property name="rotor_drag_coefficient" value="8.06428e-05" /> <!-- still to be determined -->
   <xacro:property name="rolling_moment_coefficient" value="0.000001" /> <!-- still to be determined -->
