Commit message: 2 blade blue rotors

File: rotors_description/urdf/geranos.xacro (robot description, xacro)
@@ -25,5 +25,5 @@
   <xacro:property name="rotor_offset_direction_off" value="0.274" /> <!-- [m] --> <!-- still to be determined -->
   <xacro:property name="radius_rotor_thrust_simulation" value="1" /> <!-- [m] --> <!-- radius or durchmesser -->
-  <xacro:property name="radius_rotor_direction_simulation" value="1" /> <!-- [m] --> <!-- radius or durchmesser -->
+  <xacro:property name="radius_rotor_direction_simulation" value="0.283333" /> <!-- [m] --> <!-- radius or durchmesser -->
   <xacro:property name="radius_rotor_thrust_meter" value="0.2286" /> <!-- [m] --> <!-- radius -->
   <xacro:property name="radius_rotor_direction_meter" value="0.06477" /> <!-- [m] --> <!-- radius -->

File: rotors_description/urdf/multirotor_base.xacro (robot description, xacro)
@@ -48,5 +48,5 @@
       </inertial>
       <visual>
-        <origin xyz="0.001 0 0" rpy="0 0 0" />
+        <origin xyz="0 0 0" rpy="0 0 0" />
         <geometry>
           <xacro:if value="${use_mesh_file}">
@@ -158,5 +158,5 @@
           </xacro:if>
           <xacro:unless value="${use_own_mesh}">
-            <mesh filename="package://rotors_description/meshes/geranos_direction_${direction}.dae"
+            <mesh filename="package://rotors_description/meshes/geranos_prop_${direction}.dae"
               scale="${radius_rotor} ${radius_rotor} ${radius_rotor}" /> <!-- The propeller meshes have a radius of 1m -->
             <!-- <box size="${2*radius_rotor} 0.01 0.005"/> -->
@@ -218,5 +218,5 @@
           </xacro:if>
           <xacro:unless value="${use_own_mesh}">
-            <mesh filename="package://rotors_description/meshes/geranos_direction_${direction}.dae"
+            <mesh filename="package://rotors_description/meshes/geranos_prop_${direction}.dae"
               scale="${radius_rotor} ${radius_rotor} ${radius_rotor}" /> <!-- The propeller meshes have a radius of 1m -->
             <!-- <box size="${2*radius_rotor} 0.01 0.005"/> -->
@@ -278,5 +278,5 @@
           </xacro:if>
           <xacro:unless value="${use_own_mesh}">
-            <mesh filename="package://rotors_description/meshes/geranos_direction_${direction}.dae"
+            <mesh filename="package://rotors_description/meshes/geranos_prop_${direction}.dae"
               scale="${radius_rotor} ${radius_rotor} ${radius_rotor}" /> <!-- The propeller meshes have a radius of 1m -->
             <!-- <box size="${2*radius_rotor} 0.01 0.005"/> -->
@@ -338,5 +338,5 @@
           </xacro:if>
           <xacro:unless value="${use_own_mesh}">
-            <mesh filename="package://rotors_description/meshes/geranos_direction_${direction}.dae"
+            <mesh filename="package://rotors_description/meshes/geranos_prop_${direction}.dae"
               scale="${radius_rotor} ${radius_rotor} ${radius_rotor}" /> <!-- The propeller meshes have a radius of 1m -->
             <!-- <box size="${2*radius_rotor} 0.01 0.005"/> -->

Commit message: deleted some notes

File: rotors_description/urdf/geranos.xacro (robot description, xacro)
@@ -8,5 +8,5 @@
   <xacro:property name="use_mesh_file" value="true" />
   <xacro:property name="mesh_file" value="package://rotors_description/meshes/geranos_finalprototyp1.dae" />
-  <xacro:property name="mass" value="5.0" /> <!-- [kg] --> <!-- still to be determined -->
+  <xacro:property name="mass" value="5.0" /> <!-- [kg] -->
   <xacro:property name="body_width" value="0.820" /> <!-- [m] -->
   <xacro:property name="big_rotor_x" value="0.44017" /> <!-- [m] -->
@@ -19,30 +19,30 @@
   <xacro:property name="side_length_two" value="0.3" /> <!-- [m] -->
   <xacro:property name="body_height" value="0.736" /> <!-- [m] -->
-  <xacro:property name="mass_rotor_thrust" value="0.05" /> <!-- [kg] --> <!-- still to be determined -->
-  <xacro:property name="mass_rotor_direction" value="0.005" /> <!-- [kg] --> <!-- still to be determined -->
-  <xacro:property name="rotor_offset_thrust" value="0.13" /> <!-- [m] --> <!-- still to be determined -->
-  <xacro:property name="rotor_offset_direction" value="0.267" /> <!-- [m] --> <!-- still to be determined -->
-  <xacro:property name="rotor_offset_direction_off" value="0.274" /> <!-- [m] --> <!-- still to be determined -->
-  <xacro:property name="radius_rotor_thrust_simulation" value="1" /> <!-- [m] --> <!-- radius or durchmesser -->
-  <xacro:property name="radius_rotor_direction_simulation" value="0.283333" /> <!-- [m] --> <!-- radius or durchmesser -->
+  <xacro:property name="mass_rotor_thrust" value="0.05" /> <!-- [kg] -->
+  <xacro:property name="mass_rotor_direction" value="0.005" /> <!-- [kg] -->
+  <xacro:property name="rotor_offset_thrust" value="0.13" /> <!-- [m] -->
+  <xacro:property name="rotor_offset_direction" value="0.267" /> <!-- [m] -->
+  <xacro:property name="rotor_offset_direction_off" value="0.274" /> <!-- [m] -->
+  <xacro:property name="radius_rotor_thrust_simulation" value="1" /> <!-- [m] --> <!-- ratio -->
+  <xacro:property name="radius_rotor_direction_simulation" value="0.283333" /> <!-- [m] --> <!-- ratio -->
   <xacro:property name="radius_rotor_thrust_meter" value="0.2286" /> <!-- [m] --> <!-- radius -->
   <xacro:property name="radius_rotor_direction_meter" value="0.06477" /> <!-- [m] --> <!-- radius -->
-  <xacro:property name="motor_constant" value="8.54858e-06" /> <!-- [kg.m/s^2] -->  <!-- still to be determined -->
-  <xacro:property name="moment_constant" value="0.016" /> <!-- [m] --> <!-- still to be determined -->
-  <xacro:property name="time_constant_up" value="0.0125" /> <!-- [s] --> <!-- still to be determined -->
-  <xacro:property name="time_constant_down" value="0.025" /> <!-- [s] --> <!-- still to be determined -->
-  <xacro:property name="max_rot_velocity_thrust" value="2000" /> <!-- [rad/s] --> <!-- still to be determined -->
-  <xacro:property name="max_rot_velocity_direction" value="2000" /> <!-- [rad/s] --> <!-- still to be determined -->
-  <xacro:property name="rotor_drag_coefficient" value="8.06428e-05" /> <!-- still to be determined -->
-  <xacro:property name="rolling_moment_coefficient" value="0.000001" /> <!-- still to be determined -->
+  <xacro:property name="motor_constant" value="8.54858e-06" /> <!-- [kg.m/s^2] -->
+  <xacro:property name="moment_constant" value="0.016" /> <!-- [m] -->
+  <xacro:property name="time_constant_up" value="0.0125" /> <!-- [s] -->
+  <xacro:property name="time_constant_down" value="0.025" /> <!-- [s] -->
+  <xacro:property name="max_rot_velocity_thrust" value="2000" /> <!-- [rad/s] -->
+  <xacro:property name="max_rot_velocity_direction" value="2000" /> <!-- [rad/s] -->
+  <xacro:property name="rotor_drag_coefficient" value="8.06428e-05" />
+  <xacro:property name="rolling_moment_coefficient" value="0.000001" />
   <!-- Property Blocks -->
-  <xacro:property name="body_inertia"> <!-- still to be determined -->
+  <xacro:property name="body_inertia">
     <inertia ixx="0.06" ixy="0.0" ixz="0.0" iyy="0.10" iyz="0.0" izz="0.15" /> <!-- [kg.m^2] [kg.m^2] [kg.m^2] [kg.m^2] [kg.m^2] [kg.m^2] -->
   </xacro:property>
   <!-- inertia of a single rotor, assuming it is a cuboid. Height=3mm, width=15mm -->
-  <xacro:property name="rotor_inertia_thrust"> <!-- still to be determined -->
+  <xacro:property name="rotor_inertia_thrust">
     <xacro:box_inertia x="${radius_rotor_thrust_meter}" y="0.015" z="0.003" mass="${mass_rotor_thrust*rotor_velocity_slowdown_thrust}" />
   </xacro:property>
-  <xacro:property name="rotor_inertia_direction"> <!-- still to be determined -->
+  <xacro:property name="rotor_inertia_direction">
     <xacro:box_inertia x="${radius_rotor_direction_meter}" y="0.015" z="0.003" mass="${mass_rotor_direction*rotor_velocity_slowdown_direction}" />
   </xacro:property>

Commit message: changed motor and force constants

File: rotors_description/urdf/geranos.xacro (robot description, xacro)
@@ -28,6 +28,8 @@
   <xacro:property name="radius_rotor_thrust_meter" value="0.2286" /> <!-- [m] --> <!-- radius -->
   <xacro:property name="radius_rotor_direction_meter" value="0.06477" /> <!-- [m] --> <!-- radius -->
-  <xacro:property name="motor_constant" value="8.54858e-06" /> <!-- [kg.m/s^2] -->
-  <xacro:property name="moment_constant" value="0.016" /> <!-- [m] -->
+  <xacro:property name="motor_constant_thrust" value="8.58307e-05" /> <!-- [kg.m/s^2] -->
+  <xacro:property name="motor_constant_direction" value="1.21542e-06" /> <!-- [kg.m/s^2] -->
+  <xacro:property name="moment_constant_thrust" value="0.0214167" /> <!-- [m] -->
+  <xacro:property name="moment_constant_direction" value="0.011378057" /> <!-- [m] -->
   <xacro:property name="time_constant_up" value="0.0125" /> <!-- [s] -->
   <xacro:property name="time_constant_down" value="0.025" /> <!-- [s] -->
@@ -65,6 +67,6 @@
     suffix="front_right"
     direction="ccw"
-    motor_constant="${motor_constant}"
-    moment_constant="${moment_constant}"
+    motor_constant="${motor_constant_thrust}"
+    moment_constant="${moment_constant_thrust}"
     parent="${namespace}/base_link"
     mass_rotor="${mass_rotor_thrust}"
@@ -86,6 +88,6 @@
     suffix="back_left"
     direction="ccw"
-    motor_constant="${motor_constant}"
-    moment_constant="${moment_constant}"
+    motor_constant="${motor_constant_thrust}"
+    moment_constant="${moment_constant_thrust}"
     parent="${namespace}/base_link"
     mass_rotor="${mass_rotor_thrust}"
@@ -106,6 +108,6 @@
     suffix="back_right"
     direction="cw"
-    motor_constant="${motor_constant}"
-    moment_constant="${moment_constant}"
+    motor_constant="${motor_constant_thrust}"
+    moment_constant="${moment_constant_thrust}"
     parent="${namespace}/base_link"
     mass_rotor="${mass_rotor_thrust}"
@@ -126,6 +128,6 @@
     suffix="front_left"
     direction="cw"
-    motor_constant="${motor_constant}"
-    moment_constant="${moment_constant}"
+    motor_constant="${motor_constant_thrust}"
+    moment_constant="${moment_constant_thrust}"
     parent="${namespace}/base_link"
     mass_rotor="${mass_rotor_thrust}"
@@ -146,6 +148,6 @@
     suffix="direction_front"
     direction="cw"
-    motor_constant="${motor_constant}"
-    moment_constant="${moment_constant}"
+    motor_constant="${motor_constant_direction}"
+    moment_constant="${moment_constant_direction}"
     parent="${namespace}/base_link"
     mass_rotor="${mass_rotor_direction}"
@@ -166,6 +168,6 @@
     suffix="direciton_back"
     direction="cw"
-    motor_constant="${motor_constant}"
-    moment_constant="${moment_constant}"
+    motor_constant="${motor_constant_direction}"
+    moment_constant="${moment_constant_direction}"
     parent="${namespace}/base_link"
     mass_rotor="${mass_rotor_direction}"
@@ -186,6 +188,6 @@
     suffix="direction_right"
     direction="ccw"
-    motor_constant="${motor_constant}"
-    moment_constant="${moment_constant}"
+    motor_constant="${motor_constant_direction}"
+    moment_constant="${moment_constant_direction}"
     parent="${namespace}/base_link"
     mass_rotor="${mass_rotor_direction}"
@@ -206,6 +208,6 @@
     suffix="direction_left"
     direction="ccw"
-    motor_constant="${motor_constant}"
-    moment_constant="${moment_constant}"
+    motor_constant="${motor_constant_direction}"
+    moment_constant="${moment_constant_direction}"
     parent="${namespace}/base_link"
     mass_rotor="${mass_rotor_direction}"

Commit message: changes to actual force constants

File: rotors_description/urdf/geranos.xacro (robot description, xacro)
@@ -28,14 +28,16 @@
   <xacro:property name="radius_rotor_thrust_meter" value="0.2286" /> <!-- [m] --> <!-- radius -->
   <xacro:property name="radius_rotor_direction_meter" value="0.06477" /> <!-- [m] --> <!-- radius -->
-  <xacro:property name="motor_constant" value="8.54858e-06" /> <!-- [kg.m/s^2] -->
-  <xacro:property name="moment_constant" value="0.016" /> <!-- [m] -->
+  <xacro:property name="motor_constant_thrust" value="8.58307e-05" /> <!-- [kg.m/s^2] -->
+  <xacro:property name="motor_constant_direction" value="1.21542e-06" /> <!-- [kg.m/s^2] -->  <!--1.21542e-06-->
+  <xacro:property name="moment_constant_thrust" value="0.02141697" /> <!-- [m] -->
+  <xacro:property name="moment_constant_direction" value="0.011378057" /> <!-- [m] -->        <!--0.011378057-->
   <xacro:property name="time_constant_up" value="0.0125" /> <!-- [s] -->
   <xacro:property name="time_constant_down" value="0.025" /> <!-- [s] -->
-  <xacro:property name="max_rot_velocity_thrust" value="2000" /> <!-- [rad/s] -->
-  <xacro:property name="max_rot_velocity_direction" value="2000" /> <!-- [rad/s] -->
+  <xacro:property name="max_rot_velocity_thrust" value="2500" /> <!-- [rad/s] -->
+  <xacro:property name="max_rot_velocity_direction" value="2500" /> <!-- [rad/s] -->
   <xacro:property name="rotor_drag_coefficient" value="8.06428e-05" />
   <xacro:property name="rolling_moment_coefficient" value="0.000001" />
   <!-- Property Blocks -->
-  <xacro:property name="body_inertia">
+  <xacro:property name="body_inertia"> <!-- still to be determined -->
     <inertia ixx="0.06" ixy="0.0" ixz="0.0" iyy="0.10" iyz="0.0" izz="0.15" /> <!-- [kg.m^2] [kg.m^2] [kg.m^2] [kg.m^2] [kg.m^2] [kg.m^2] -->
   </xacro:property>
@@ -65,6 +67,6 @@
     suffix="front_right"
     direction="ccw"
-    motor_constant="${motor_constant}"
-    moment_constant="${moment_constant}"
+    motor_constant="${motor_constant_thrust}"
+    moment_constant="${moment_constant_thrust}"
     parent="${namespace}/base_link"
     mass_rotor="${mass_rotor_thrust}"
@@ -86,6 +88,6 @@
     suffix="back_left"
     direction="ccw"
-    motor_constant="${motor_constant}"
-    moment_constant="${moment_constant}"
+    motor_constant="${motor_constant_thrust}"
+    moment_constant="${moment_constant_thrust}"
     parent="${namespace}/base_link"
     mass_rotor="${mass_rotor_thrust}"
@@ -106,6 +108,6 @@
     suffix="back_right"
     direction="cw"
-    motor_constant="${motor_constant}"
-    moment_constant="${moment_constant}"
+    motor_constant="${motor_constant_thrust}"
+    moment_constant="${moment_constant_thrust}"
     parent="${namespace}/base_link"
     mass_rotor="${mass_rotor_thrust}"
@@ -126,6 +128,6 @@
     suffix="front_left"
     direction="cw"
-    motor_constant="${motor_constant}"
-    moment_constant="${moment_constant}"
+    motor_constant="${motor_constant_thrust}"
+    moment_constant="${moment_constant_thrust}"
     parent="${namespace}/base_link"
     mass_rotor="${mass_rotor_thrust}"
@@ -146,6 +148,6 @@
     suffix="direction_front"
     direction="cw"
-    motor_constant="${motor_constant}"
-    moment_constant="${moment_constant}"
+    motor_constant="${motor_constant_direction}"
+    moment_constant="${moment_constant_direction}"
     parent="${namespace}/base_link"
     mass_rotor="${mass_rotor_direction}"
@@ -166,6 +168,6 @@
     suffix="direciton_back"
     direction="cw"
-    motor_constant="${motor_constant}"
-    moment_constant="${moment_constant}"
+    motor_constant="${motor_constant_direction}"
+    moment_constant="${moment_constant_direction}"
     parent="${namespace}/base_link"
     mass_rotor="${mass_rotor_direction}"
@@ -186,6 +188,6 @@
     suffix="direction_right"
     direction="ccw"
-    motor_constant="${motor_constant}"
-    moment_constant="${moment_constant}"
+    motor_constant="${motor_constant_direction}"
+    moment_constant="${moment_constant_direction}"
     parent="${namespace}/base_link"
     mass_rotor="${mass_rotor_direction}"
@@ -206,6 +208,6 @@
     suffix="direction_left"
     direction="ccw"
-    motor_constant="${motor_constant}"
-    moment_constant="${moment_constant}"
+    motor_constant="${motor_constant_direction}"
+    moment_constant="${moment_constant_direction}"
     parent="${namespace}/base_link"
     mass_rotor="${mass_rotor_direction}"

Commit message: edited weird numbers in geranos.xacro

File: rotors_description/urdf/geranos.xacro (robot description, xacro)
@@ -12,7 +12,6 @@
   <xacro:property name="big_rotor_x" value="0.44017" /> <!-- [m] -->
   <xacro:property name="big_rotor_y" value="0.4098" /> <!-- [m] -->
-  <xacro:property name="small_rotor_x" value="0.463" /> <!-- [m] -->
-  <xacro:property name="small_rotor_y" value="0.363" /> <!-- [m] -->
-  <xacro:property name="small_rotor_x_off" value="0.4547" /> <!-- [m] -->
+  <xacro:property name="small_rotor_x" value="0.4481" /> <!-- [m] -->
+  <xacro:property name="small_rotor_y" value="0.34809" /> <!-- [m] -->
   <xacro:property name="half_body_width" value="0.3" /> <!-- [m] -->
   <xacro:property name="side_length_one" value="0.2" /> <!-- [m] -->
@@ -22,6 +21,5 @@
   <xacro:property name="mass_rotor_direction" value="0.005" /> <!-- [kg] -->
   <xacro:property name="rotor_offset_thrust" value="0.13" /> <!-- [m] -->
-  <xacro:property name="rotor_offset_direction" value="0.267" /> <!-- [m] -->
-  <xacro:property name="rotor_offset_direction_off" value="0.274" /> <!-- [m] -->
+  <xacro:property name="rotor_offset_direction" value="0.26005" /> <!-- [m] -->
   <xacro:property name="radius_rotor_thrust_simulation" value="1" /> <!-- [m] --> <!-- ratio -->
   <xacro:property name="radius_rotor_direction_simulation" value="0.283333" /> <!-- [m] --> <!-- ratio -->
@@ -182,5 +180,5 @@
     use_own_mesh="false"
     mesh="">
-    <origin xyz="-${small_rotor_x_off} 0 ${rotor_offset_direction_off}" rpy="0 0.837758 0" />
+    <origin xyz="-${small_rotor_x} 0 ${rotor_offset_direction}" rpy="0 0.837758 0" />
     <xacro:insert_block name="rotor_inertia_direction" />
   </xacro:direction_b_rotor>

Commit message: added python exp for angle

File: rotors_description/urdf/geranos.xacro (robot description, xacro)
@@ -28,4 +28,7 @@
   <xacro:property name="radius_rotor_thrust_meter" value="0.2286" /> <!-- [m] --> <!-- radius -->
   <xacro:property name="radius_rotor_direction_meter" value="0.06477" /> <!-- [m] --> <!-- radius -->
+  <xacro:property name="angle" value="${48/180*pi}" /> <!-- [rad] --> <!--  -->
+  <xacro:property name="sin_angle" value="0.5" /> <!-- [m] --> <!--  -->
+  <xacro:property name="cos_angle" value="0.5" /> <!-- [m] --> <!--  -->
   <xacro:property name="motor_constant_thrust" value="8.58307e-05" /> <!-- [kg.m/s^2] -->
   <xacro:property name="motor_constant_direction" value="1.21542e-06" /> <!-- [kg.m/s^2] -->  <!--1.21542e-06-->
@@ -162,5 +165,5 @@
     use_own_mesh="false"
     mesh="">
-    <origin xyz="${small_rotor_x}  0 ${rotor_offset_direction}" rpy="0 -0.837758 0" />
+    <origin xyz="${small_rotor_x}  0 ${rotor_offset_direction}" rpy="0 -${angle} 0" />
     <xacro:insert_block name="rotor_inertia_direction" />
   </xacro:direction_f_rotor>
@@ -182,5 +185,5 @@
     use_own_mesh="false"
     mesh="">
-    <origin xyz="-${small_rotor_x_off} 0 ${rotor_offset_direction_off}" rpy="0 0.837758 0" />
+    <origin xyz="-${small_rotor_x_off} 0 ${rotor_offset_direction_off}" rpy="0 ${angle} 0" />
     <xacro:insert_block name="rotor_inertia_direction" />
   </xacro:direction_b_rotor>
@@ -202,5 +205,5 @@
     use_own_mesh="false"
     mesh="">
-    <origin xyz="0 ${small_rotor_y}  ${rotor_offset_direction}" rpy="0.837758 0 0" />
+    <origin xyz="0 ${small_rotor_y}  ${rotor_offset_direction}" rpy="${angle} 0 0" />
     <xacro:insert_block name="rotor_inertia_direction" />
   </xacro:direction_r_rotor>
@@ -222,5 +225,5 @@
     use_own_mesh="false"
     mesh="">
-    <origin xyz="0 -${small_rotor_y}  ${rotor_offset_direction}" rpy="-0.837758 0 0" />
+    <origin xyz="0 -${small_rotor_y}  ${rotor_offset_direction}" rpy="-${angle} 0 0" />
     <xacro:insert_block name="rotor_inertia_direction" />
   </xacro:direction_l_rotor>

Commit message: added dependency on angle

File: rotors_description/urdf/geranos.xacro (robot description, xacro)
@@ -10,8 +10,9 @@
   <xacro:property name="mass" value="5.0" /> <!-- [kg] -->
   <xacro:property name="body_width" value="0.820" /> <!-- [m] -->
+  <xacro:property name="angle" value="${48/180*pi}" /> <!-- [rad] -->
   <xacro:property name="big_rotor_x" value="0.44017" /> <!-- [m] -->
   <xacro:property name="big_rotor_y" value="0.4098" /> <!-- [m] -->
-  <xacro:property name="small_rotor_x" value="0.4481" /> <!-- [m] -->
-  <xacro:property name="small_rotor_y" value="0.34809" /> <!-- [m] -->
+  <xacro:property name="small_rotor_x" value="${0.331 + 0.175 * cos(angle)}" /> <!-- [m] -->
+  <xacro:property name="small_rotor_y" value="${0.231 + 0.175 * sin(angle)}" /> <!-- [m] -->
   <xacro:property name="half_body_width" value="0.3" /> <!-- [m] -->
   <xacro:property name="side_length_one" value="0.2" /> <!-- [m] -->
@@ -21,5 +22,5 @@
   <xacro:property name="mass_rotor_direction" value="0.005" /> <!-- [kg] -->
   <xacro:property name="rotor_offset_thrust" value="0.13" /> <!-- [m] -->
-  <xacro:property name="rotor_offset_direction" value="0.26005" /> <!-- [m] -->
+  <xacro:property name="rotor_offset_direction" value="0.13 + 0.175 * sin(angle)" /> <!-- [m] -->
   <xacro:property name="radius_rotor_thrust_simulation" value="1" /> <!-- [m] --> <!-- ratio -->
   <xacro:property name="radius_rotor_direction_simulation" value="0.283333" /> <!-- [m] --> <!-- ratio -->
@@ -38,5 +39,5 @@
   <!-- Property Blocks -->
   <xacro:property name="body_inertia"> <!-- still to be determined -->
-    <inertia ixx="0.06" ixy="0.0" ixz="0.0" iyy="0.10" iyz="0.0" izz="0.15" /> <!-- [kg.m^2] [kg.m^2] [kg.m^2] [kg.m^2] [kg.m^2] [kg.m^2] -->
+    <inertia ixx="0.6664" ixy="-0.0339" ixz="0.0009" iyy="0.4543" iyz="-0.0003" izz="0.2822" /> <!-- [kg.m^2] [kg.m^2] [kg.m^2] [kg.m^2] [kg.m^2] [kg.m^2] -->
   </xacro:property>
   <!-- inertia of a single rotor, assuming it is a cuboid. Height=3mm, width=15mm -->
@@ -160,5 +161,5 @@
     use_own_mesh="false"
     mesh="">
-    <origin xyz="${small_rotor_x}  0 ${rotor_offset_direction}" rpy="0 -0.837758 0" />
+    <origin xyz="${small_rotor_x}  0 ${rotor_offset_direction}" rpy="0 -${angle} 0" />
     <xacro:insert_block name="rotor_inertia_direction" />
   </xacro:direction_f_rotor>
@@ -180,5 +181,5 @@
     use_own_mesh="false"
     mesh="">
-    <origin xyz="-${small_rotor_x} 0 ${rotor_offset_direction}" rpy="0 0.837758 0" />
+    <origin xyz="-${small_rotor_x} 0 ${rotor_offset_direction}" rpy="0 ${angle} 0" />
     <xacro:insert_block name="rotor_inertia_direction" />
   </xacro:direction_b_rotor>
@@ -200,5 +201,5 @@
     use_own_mesh="false"
     mesh="">
-    <origin xyz="0 ${small_rotor_y}  ${rotor_offset_direction}" rpy="0.837758 0 0" />
+    <origin xyz="0 ${small_rotor_y}  ${rotor_offset_direction}" rpy="${angle} 0 0" />
     <xacro:insert_block name="rotor_inertia_direction" />
   </xacro:direction_r_rotor>
@@ -220,5 +221,5 @@
     use_own_mesh="false"
     mesh="">
-    <origin xyz="0 -${small_rotor_y}  ${rotor_offset_direction}" rpy="-0.837758 0 0" />
+    <origin xyz="0 -${small_rotor_y}  ${rotor_offset_direction}" rpy="-${angle} 0 0" />
     <xacro:insert_block name="rotor_inertia_direction" />
   </xacro:direction_l_rotor>
