Commit message: bug fix

File: rotors_description/urdf/geranos.xacro (robot description, xacro)
@@ -10,9 +10,9 @@
   <xacro:property name="mass" value="5.0" /> <!-- [kg] -->
   <xacro:property name="body_width" value="0.820" /> <!-- [m] -->
-  <xacro:property name="angle" value="${48/180*pi}" /> <!-- [rad] -->
+  <xacro:property name="angle" value="${30/180*pi}" /> <!-- [rad] -->
   <xacro:property name="big_rotor_x" value="0.44017" /> <!-- [m] -->
   <xacro:property name="big_rotor_y" value="0.4098" /> <!-- [m] -->
-  <xacro:property name="small_rotor_x" value="${0.331 + 0.175 * cos(angle)}" /> <!-- [m] -->
-  <xacro:property name="small_rotor_y" value="${0.231 + 0.175 * sin(angle)}" /> <!-- [m] -->
+  <xacro:property name="small_rotor_x" value="${0.331+0.175*cos(angle)}" /> <!-- [m] -->
+  <xacro:property name="small_rotor_y" value="${0.231+0.175*sin(angle)}" /> <!-- [m] -->
   <xacro:property name="half_body_width" value="0.3" /> <!-- [m] -->
   <xacro:property name="side_length_one" value="0.2" /> <!-- [m] -->
@@ -22,5 +22,5 @@
   <xacro:property name="mass_rotor_direction" value="0.005" /> <!-- [kg] -->
   <xacro:property name="rotor_offset_thrust" value="0.13" /> <!-- [m] -->
-  <xacro:property name="rotor_offset_direction" value="0.13 + 0.175 * sin(angle)" /> <!-- [m] -->
+  <xacro:property name="rotor_offset_direction" value="${0.13+0.175*sin(angle)}" /> <!-- [m] -->
   <xacro:property name="radius_rotor_thrust_simulation" value="1" /> <!-- [m] --> <!-- ratio -->
   <xacro:property name="radius_rotor_direction_simulation" value="0.283333" /> <!-- [m] --> <!-- ratio -->

Commit message: Changed urdf to 90degrees tilted rotors!

File: rotors_description/urdf/geranos.xacro (robot description, xacro)
@@ -10,9 +10,9 @@
   <xacro:property name="mass" value="5.0" /> <!-- [kg] -->
   <xacro:property name="body_width" value="0.820" /> <!-- [m] -->
-  <xacro:property name="angle" value="${30/180*pi}" /> <!-- [rad] -->
+  <xacro:property name="angle" value="${0/180*pi}" /> <!-- [rad] -->
   <xacro:property name="big_rotor_x" value="0.44017" /> <!-- [m] -->
   <xacro:property name="big_rotor_y" value="0.4098" /> <!-- [m] -->
   <xacro:property name="small_rotor_x" value="${0.331+0.175*cos(angle)}" /> <!-- [m] -->
-  <xacro:property name="small_rotor_y" value="${0.231+0.175*sin(angle)}" /> <!-- [m] -->
+  <xacro:property name="small_rotor_y" value="${0.231+0.175*cos(angle)}" /> <!-- [m] -->
   <xacro:property name="half_body_width" value="0.3" /> <!-- [m] -->
   <xacro:property name="side_length_one" value="0.2" /> <!-- [m] -->
@@ -161,5 +161,5 @@
     use_own_mesh="false"
     mesh="">
-    <origin xyz="${small_rotor_x}  0 ${rotor_offset_direction}" rpy="0 -${angle} 0" />
+    <origin xyz="${small_rotor_x}  0 ${rotor_offset_direction}" rpy="0 1.5708 0" />
     <xacro:insert_block name="rotor_inertia_direction" />
   </xacro:direction_f_rotor>
@@ -181,5 +181,5 @@
     use_own_mesh="false"
     mesh="">
-    <origin xyz="-${small_rotor_x} 0 ${rotor_offset_direction}" rpy="0 ${angle} 0" />
+    <origin xyz="-${small_rotor_x} 0 ${rotor_offset_direction}" rpy="0 -1.5708 0" />
     <xacro:insert_block name="rotor_inertia_direction" />
   </xacro:direction_b_rotor>
@@ -201,5 +201,5 @@
     use_own_mesh="false"
     mesh="">
-    <origin xyz="0 ${small_rotor_y}  ${rotor_offset_direction}" rpy="${angle} 0 0" />
+    <origin xyz="0 ${small_rotor_y}  ${rotor_offset_direction}" rpy="-1.5708 0 0" />
     <xacro:insert_block name="rotor_inertia_direction" />
   </xacro:direction_r_rotor>
@@ -221,5 +221,5 @@
     use_own_mesh="false"
     mesh="">
-    <origin xyz="0 -${small_rotor_y}  ${rotor_offset_direction}" rpy="-${angle} 0 0" />
+    <origin xyz="0 -${small_rotor_y}  ${rotor_offset_direction}" rpy="1.5708 0 0" />
     <xacro:insert_block name="rotor_inertia_direction" />
   </xacro:direction_l_rotor>

Commit message: Changed angles corresponding to atlas

File: rotors_description/urdf/geranos.xacro (robot description, xacro)
@@ -161,5 +161,5 @@
     use_own_mesh="false"
     mesh="">
-    <origin xyz="${small_rotor_x}  0 ${rotor_offset_direction}" rpy="0 1.5708 0" />
+    <origin xyz="${small_rotor_x}  0 ${rotor_offset_direction}" rpy="0 -1.5708 0" />
     <xacro:insert_block name="rotor_inertia_direction" />
   </xacro:direction_f_rotor>
@@ -181,5 +181,5 @@
     use_own_mesh="false"
     mesh="">
-    <origin xyz="-${small_rotor_x} 0 ${rotor_offset_direction}" rpy="0 -1.5708 0" />
+    <origin xyz="-${small_rotor_x} 0 ${rotor_offset_direction}" rpy="0 1.5708 0" />
     <xacro:insert_block name="rotor_inertia_direction" />
   </xacro:direction_b_rotor>
@@ -201,5 +201,5 @@
     use_own_mesh="false"
     mesh="">
-    <origin xyz="0 ${small_rotor_y}  ${rotor_offset_direction}" rpy="-1.5708 0 0" />
+    <origin xyz="0 ${small_rotor_y}  ${rotor_offset_direction}" rpy="1.5708 0 0" />
     <xacro:insert_block name="rotor_inertia_direction" />
   </xacro:direction_r_rotor>
@@ -221,5 +221,5 @@
     use_own_mesh="false"
     mesh="">
-    <origin xyz="0 -${small_rotor_y}  ${rotor_offset_direction}" rpy="1.5708 0 0" />
+    <origin xyz="0 -${small_rotor_y}  ${rotor_offset_direction}" rpy="-1.5708 0 0" />
     <xacro:insert_block name="rotor_inertia_direction" />
   </xacro:direction_l_rotor>
