Commit message: local test branch. Boreas setup the same way as atlas

File: rotors_description/urdf/boreas.xacro (robot description, xacro)
@@ -4,5 +4,5 @@
   <xacro:property name="namespace" value="$(arg namespace)" />
   <xacro:property name="rotor_velocity_slowdown_thrust" value="10" />
-  <xacro:property name="rotor_velocity_slowdown_auxiliary" value="4" />
+  <xacro:property name="rotor_velocity_slowdown_direction" value="4" />
   <xacro:property name="rotor_velocity_slowdown_sim" value="10" />
   <xacro:property name="use_mesh_file" value="true" />
@@ -17,19 +17,19 @@
   <xacro:property name="rotation" value="3.14" /> <!-- 180 degrees -->
   <xacro:property name="z_offset" value="0.024" /> <!-- [m] -->
-  <xacro:property name="z_offset_auxiliary" value="-0.0285" /> <!-- [m] -->#
+  <xacro:property name="z_offset_direction" value="-0.0285" /> <!-- [m] -->
   <xacro:property name="mass_rotor_thrust" value="0.05" /> <!-- [kg] -->
-  <xacro:property name="mass_rotor_auxiliary" value="0.01" /> <!-- [kg] -->
+  <xacro:property name="mass_rotor_direction" value="0.01" /> <!-- [kg] -->
   <xacro:property name="radius_rotor_thrust_meter" value="0.2286" /> <!-- radius in [m] -->
-  <xacro:property name="radius_rotor_auxiliary_meter" value="0.06477" /> <!-- radius in [m] -->
+  <xacro:property name="radius_rotor_direction_meter" value="0.06477" /> <!-- radius in [m] -->
   <xacro:property name="radius_rotor_thrust_simulation" value="1" />  <!-- ratio -->
-  <xacro:property name="radius_rotor_auxiliary_simulation" value="0.283" />  <!-- ratio -->
+  <xacro:property name="radius_rotor_direction_simulation" value="0.283" />  <!-- ratio -->
   <xacro:property name="motor_constant_thrust" value="8.58307e-05" /> <!-- [kg.m/s^2] -->
-  <xacro:property name="motor_constant_auxiliary" value="1.21542e-06" /> <!-- [kg.m/s^2] -->  <!--1.21542e-06-->
+  <xacro:property name="motor_constant_direction" value="1.21542e-06" /> <!-- [kg.m/s^2] -->  <!--1.21542e-06-->
   <xacro:property name="moment_constant_thrust" value="0.02141697" /> <!-- [m] -->
-  <xacro:property name="moment_constant_auxiliary" value="0.011378057" /> <!-- [m] -->        <!--0.011378057-->
+  <xacro:property name="moment_constant_direction" value="0.011378057" /> <!-- [m] -->        <!--0.011378057-->
   <xacro:property name="time_constant_up" value="0.0125" /> <!-- [s] -->
   <xacro:property name="time_constant_down" value="0.025" /> <!-- [s] -->
   <xacro:property name="max_rot_velocity_thrust" value="2500" /> <!-- [rad/s] -->
-  <xacro:property name="max_rot_velocity_auxiliary" value="2500" /> <!-- [rad/s] -->
+  <xacro:property name="max_rot_velocity_direction" value="2500" /> <!-- [rad/s] -->
   <xacro:property name="rotor_drag_coefficient" value="8.06428e-05" />
   <xacro:property name="rolling_moment_coefficient" value="0.000001" />
@@ -42,9 +42,9 @@
     <xacro:box_inertia x="${radius_rotor_thrust_meter}" y="0.015" z="0.003" mass="${mass_rotor_thrust*rotor_velocity_slowdown_thrust}" />
   </xacro:property>
-  <xacro:property name="rotor_inertia_auxiliary">
-    <xacro:box_inertia x="${radius_rotor_auxiliary_meter}" y="0.015" z="0.003" mass="${mass_rotor_auxiliary*rotor_velocity_slowdown_auxiliary}" />
+  <xacro:property name="rotor_inertia_direction">
+    <xacro:box_inertia x="${radius_rotor_direction_meter}" y="0.015" z="0.003" mass="${mass_rotor_direction*rotor_velocity_slowdown_direction}" />
   </xacro:property>
   <!-- Included URDF Files -->
-  <xacro:include filename="$(find rotors_description)/urdf/multirotor_base_boreas.xacro" />
+  <xacro:include filename="$(find rotors_description)/urdf/multirotor_base.xacro" />
   <!-- Instantiate multirotor_base_macro once -->
   <xacro:multirotor_base_macro
@@ -59,45 +59,4 @@
   </xacro:multirotor_base_macro>
   <!-- Instantiate rotors -->
-    <xacro:thrust_rotor
-    robot_namespace="${namespace}"
-    suffix="back_left"
-    direction="ccw"
-    motor_constant="${motor_constant_thrust}"
-    moment_constant="${moment_constant_thrust}"
-    parent="${namespace}/base_link"
-    mass_rotor="${mass_rotor_thrust}"
-    radius_rotor="${radius_rotor_thrust_simulation}"
-    time_constant_up="${time_constant_up}"
-    time_constant_down="${time_constant_down}"
-    max_rot_velocity="${max_rot_velocity_thrust}"
-    motor_number="0"
-    rotor_drag_coefficient="${rotor_drag_coefficient}"
-    rolling_moment_coefficient="${rolling_moment_coefficient}"
-    color="Red"
-    use_own_mesh="false"
-    mesh="">
-    <origin xyz="-${thrust_x} -${thrust_y} ${z_offset}" rpy="0 0 0" />
-    <xacro:insert_block name="rotor_inertia_thrust" />
-  </xacro:thrust_rotor>
-  <xacro:thrust_rotor robot_namespace="${namespace}"
-    suffix="back_right"
-    direction="cw"
-    motor_constant="${motor_constant_thrust}"
-    moment_constant="${moment_constant_thrust}"
-    parent="${namespace}/base_link"
-    mass_rotor="${mass_rotor_thrust}"
-    radius_rotor="${radius_rotor_thrust_simulation}"
-    time_constant_up="${time_constant_up}"
-    time_constant_down="${time_constant_down}"
-    max_rot_velocity="${max_rot_velocity_thrust}"
-    motor_number="1"
-    rotor_drag_coefficient="${rotor_drag_coefficient}"
-    rolling_moment_coefficient="${rolling_moment_coefficient}"
-    color="Red"
-    use_own_mesh="false"
-    mesh="">
-    <origin xyz="-${thrust_x} ${thrust_y} ${z_offset}" rpy="0 0 0" />
-    <xacro:insert_block name="rotor_inertia_thrust" />
-  </xacro:thrust_rotor>
   <xacro:thrust_rotor
     robot_namespace="${namespace}"
@@ -121,4 +80,45 @@
     <xacro:insert_block name="rotor_inertia_thrust" />
   </xacro:thrust_rotor>
+  <xacro:thrust_rotor
+    robot_namespace="${namespace}"
+    suffix="back_left"
+    direction="ccw"
+    motor_constant="${motor_constant_thrust}"
+    moment_constant="${moment_constant_thrust}"
+    parent="${namespace}/base_link"
+    mass_rotor="${mass_rotor_thrust}"
+    radius_rotor="${radius_rotor_thrust_simulation}"
+    time_constant_up="${time_constant_up}"
+    time_constant_down="${time_constant_down}"
+    max_rot_velocity="${max_rot_velocity_thrust}"
+    motor_number="0"
+    rotor_drag_coefficient="${rotor_drag_coefficient}"
+    rolling_moment_coefficient="${rolling_moment_coefficient}"
+    color="Red"
+    use_own_mesh="false"
+    mesh="">
+    <origin xyz="-${thrust_x} -${thrust_y} ${z_offset}" rpy="0 0 0" />
+    <xacro:insert_block name="rotor_inertia_thrust" />
+  </xacro:thrust_rotor>
+  <xacro:thrust_rotor robot_namespace="${namespace}"
+    suffix="back_right"
+    direction="cw"
+    motor_constant="${motor_constant_thrust}"
+    moment_constant="${moment_constant_thrust}"
+    parent="${namespace}/base_link"
+    mass_rotor="${mass_rotor_thrust}"
+    radius_rotor="${radius_rotor_thrust_simulation}"
+    time_constant_up="${time_constant_up}"
+    time_constant_down="${time_constant_down}"
+    max_rot_velocity="${max_rot_velocity_thrust}"
+    motor_number="1"
+    rotor_drag_coefficient="${rotor_drag_coefficient}"
+    rolling_moment_coefficient="${rolling_moment_coefficient}"
+    color="Red"
+    use_own_mesh="false"
+    mesh="">
+    <origin xyz="-${thrust_x} ${thrust_y} ${z_offset}" rpy="0 0 0" />
+    <xacro:insert_block name="rotor_inertia_thrust" />
+  </xacro:thrust_rotor>
   <xacro:thrust_rotor robot_namespace="${namespace}"
     suffix="front_left"
@@ -141,16 +141,35 @@
     <xacro:insert_block name="rotor_inertia_thrust" />
   </xacro:thrust_rotor>
-  <!-- rotor number 4-->
-    <xacro:direction_x_rotor robot_namespace="${namespace}"
+<xacro:direction_f_rotor robot_namespace="${namespace}"
+    suffix="direction_front"
+    direction="cw"
+    motor_constant="${motor_constant_direction}"
+    moment_constant="${moment_constant_direction}"
+    parent="${namespace}/base_link"
+    mass_rotor="${mass_rotor_direction}"
+    radius_rotor="${radius_rotor_direction_simulation}"
+    time_constant_up="${time_constant_up}"
+    time_constant_down="${time_constant_down}"
+    max_rot_velocity="${max_rot_velocity_direction}"
+    motor_number="6"
+    rotor_drag_coefficient="${rotor_drag_coefficient}"
+    rolling_moment_coefficient="${rolling_moment_coefficient}"
+    color="Blue"
+    use_own_mesh="false"
+    mesh="">
+    <origin xyz="${auxiliary_x}  0 ${z_offset_direction}" rpy="0 -1.5708 0" />
+    <xacro:insert_block name="rotor_inertia_direction" />
+  </xacro:direction_f_rotor>
+  <xacro:direction_b_rotor robot_namespace="${namespace}"
     suffix="direciton_back"
     direction="cw"
-    motor_constant="${motor_constant_auxiliary}"
-    moment_constant="${moment_constant_auxiliary}"
-    parent="${namespace}/base_link"
-    mass_rotor="${mass_rotor_auxiliary}"
-    radius_rotor="${radius_rotor_auxiliary_simulation}"
-    time_constant_up="${time_constant_up}"
-    time_constant_down="${time_constant_down}"
-    max_rot_velocity="${max_rot_velocity_auxiliary}"
+    motor_constant="${motor_constant_direction}"
+    moment_constant="${moment_constant_direction}"
+    parent="${namespace}/base_link"
+    mass_rotor="${mass_rotor_direction}"
+    radius_rotor="${radius_rotor_direction_simulation}"
+    time_constant_up="${time_constant_up}"
+    time_constant_down="${time_constant_down}"
+    max_rot_velocity="${max_rot_velocity_direction}"
     motor_number="4"
     rotor_drag_coefficient="${rotor_drag_coefficient}"
@@ -159,19 +178,18 @@
     use_own_mesh="false"
     mesh="">
-    <origin xyz="-${auxiliary_x} 0 ${z_offset_auxiliary}" rpy="0 ${rotation} 0" />
-    <xacro:insert_block name="rotor_inertia_auxiliary" />
-  </xacro:direction_x_rotor>
-  <!-- rotor number 5-->
-  <xacro:direction_y_rotor robot_namespace="${namespace}"
+    <origin xyz="-${auxiliary_x} 0 ${z_offset_direction}" rpy="0 1.5708 0" />
+    <xacro:insert_block name="rotor_inertia_direction" />
+  </xacro:direction_b_rotor>
+  <xacro:direction_r_rotor robot_namespace="${namespace}"
     suffix="direction_right"
     direction="ccw"
-    motor_constant="${motor_constant_auxiliary}"
-    moment_constant="${moment_constant_auxiliary}"
-    parent="${namespace}/base_link"
-    mass_rotor="${mass_rotor_auxiliary}"
-    radius_rotor="${radius_rotor_auxiliary_simulation}"
-    time_constant_up="${time_constant_up}"
-    time_constant_down="${time_constant_down}"
-    max_rot_velocity="${max_rot_velocity_auxiliary}"
+    motor_constant="${motor_constant_direction}"
+    moment_constant="${moment_constant_direction}"
+    parent="${namespace}/base_link"
+    mass_rotor="${mass_rotor_direction}"
+    radius_rotor="${radius_rotor_direction_simulation}"
+    time_constant_up="${time_constant_up}"
+    time_constant_down="${time_constant_down}"
+    max_rot_velocity="${max_rot_velocity_direction}"
     motor_number="5"
     rotor_drag_coefficient="${rotor_drag_coefficient}"
@@ -180,40 +198,18 @@
     use_own_mesh="false"
     mesh="">
-    <origin xyz="0 ${auxiliary_y} ${z_offset_auxiliary}" rpy="0 0 0" />
-    <xacro:insert_block name="rotor_inertia_auxiliary" />
-  </xacro:direction_y_rotor>
-  <!-- rotor number 6-->
-  <xacro:direction_x_rotor robot_namespace="${namespace}"
-    suffix="direction_front"
-    direction="cw"
-    motor_constant="${motor_constant_auxiliary}"
-    moment_constant="${moment_constant_auxiliary}"
-    parent="${namespace}/base_link"
-    mass_rotor="${mass_rotor_auxiliary}"
-    radius_rotor="${radius_rotor_auxiliary_simulation}"
-    time_constant_up="${time_constant_up}"
-    time_constant_down="${time_constant_down}"
-    max_rot_velocity="${max_rot_velocity_auxiliary}"
-    motor_number="6"
-    rotor_drag_coefficient="${rotor_drag_coefficient}"
-    rolling_moment_coefficient="${rolling_moment_coefficient}"
-    color="Blue"
-    use_own_mesh="false"
-    mesh="">
-    <origin xyz="${auxiliary_x} 0 ${z_offset_auxiliary}" rpy="0 0 0" />
-    <xacro:insert_block name="rotor_inertia_auxiliary" />
-  </xacro:direction_x_rotor>
-  <!-- rotor number 7-->
-  <xacro:direction_y_rotor robot_namespace="${namespace}"
+    <origin xyz="0 ${auxiliary_y}  ${z_offset_direction}" rpy="1.5708 0 0" />
+    <xacro:insert_block name="rotor_inertia_direction" />
+  </xacro:direction_r_rotor>
+  <xacro:direction_l_rotor robot_namespace="${namespace}"
     suffix="direction_left"
     direction="ccw"
-    motor_constant="${motor_constant_auxiliary}"
-    moment_constant="${moment_constant_auxiliary}"
-    parent="${namespace}/base_link"
-    mass_rotor="${mass_rotor_auxiliary}"
-    radius_rotor="${radius_rotor_auxiliary_simulation}"
-    time_constant_up="${time_constant_up}"
-    time_constant_down="${time_constant_down}"
-    max_rot_velocity="${max_rot_velocity_auxiliary}"
+    motor_constant="${motor_constant_direction}"
+    moment_constant="${moment_constant_direction}"
+    parent="${namespace}/base_link"
+    mass_rotor="${mass_rotor_direction}"
+    radius_rotor="${radius_rotor_direction_simulation}"
+    time_constant_up="${time_constant_up}"
+    time_constant_down="${time_constant_down}"
+    max_rot_velocity="${max_rot_velocity_direction}"
     motor_number="7"
     rotor_drag_coefficient="${rotor_drag_coefficient}"
@@ -222,6 +218,6 @@
     use_own_mesh="false"
     mesh="">
-    <origin xyz="0 -${auxiliary_y}  ${z_offset_auxiliary}" rpy="${rotation} 0 0" />
-    <xacro:insert_block name="rotor_inertia_auxiliary" />
-  </xacro:direction_y_rotor>
+    <origin xyz="0 -${auxiliary_y}  ${z_offset_direction}" rpy="-1.5708 0 0" />
+    <xacro:insert_block name="rotor_inertia_direction" />
+  </xacro:direction_l_rotor>
 </robot>

File: rotors_description/urdf/multirotor_base.xacro (robot description, xacro)
@@ -61,5 +61,5 @@
         <origin xyz="0 0 0" rpy="0 0 0" />
         <geometry>
-          <box size="${body_width} ${body_width} ${body_height}" /> <!-- [m] [m] [m] -->
+          <mesh filename="${mesh_file}" scale="1 1 1" />
         </geometry>
       </collision>
@@ -104,9 +104,4 @@
         </geometry>
       </visual>
-      <collision>
-        <geometry>
-          <cylinder length="0.007" radius="${radius_rotor}" /> <!-- [m] -->
-        </geometry>
-      </collision>
     </link>
     <gazebo>
@@ -164,9 +159,4 @@
         </geometry>
       </visual>
-      <collision>
-        <geometry>
-          <cylinder length="0.007" radius="${radius_rotor}" /> <!-- [m] -->
-        </geometry>
-      </collision>
     </link>
     <gazebo>
@@ -224,9 +214,4 @@
         </geometry>
       </visual>
-      <collision>
-        <geometry>
-          <cylinder length="0.007" radius="${radius_rotor}" /> <!-- [m] -->
-        </geometry>
-      </collision>
     </link>
     <gazebo>
@@ -284,9 +269,4 @@
         </geometry>
       </visual>
-      <collision>
-        <geometry>
-          <cylinder length="0.007" radius="${radius_rotor}" /> <!-- [m] -->
-        </geometry>
-      </collision>
     </link>
     <gazebo>
@@ -344,9 +324,4 @@
         </geometry>
       </visual>
-      <collision>
-        <geometry>
-          <cylinder length="0.007" radius="${radius_rotor}" /> <!-- [m] -->
-        </geometry>
-      </collision>
     </link>
     <gazebo>

Commit message: Added inertia to xacro

File: rotors_description/urdf/boreas.xacro (robot description, xacro)
@@ -36,5 +36,5 @@
   <!-- Property Blocks -->
   <xacro:property name="body_inertia"> <!-- TODO -->
-    <inertia ixx="0.6664" ixy="-0.0339" ixz="0.0009" iyy="0.4543" iyz="-0.0003" izz="0.2822" /> <!-- [kg.m^2] [kg.m^2] [kg.m^2] [kg.m^2] [kg.m^2] [kg.m^2] -->
+    <inertia ixx="0.4559" ixy="0.0161" ixz="-0.0083" iyy="0.4489" iyz="0.0020" izz="0.6497" /> <!-- [kg.m^2] [kg.m^2] [kg.m^2] [kg.m^2] [kg.m^2] [kg.m^2] -->
   </xacro:property>
     <!-- inertia of a single rotor, assuming it is a cuboid. Height=3mm, width=15mm -->

Commit message: changes to account for CoM offset in simulation

File: rotors_description/urdf/boreas.xacro (robot description, xacro)
@@ -8,5 +8,5 @@
   <xacro:property name="use_mesh_file" value="true" />
   <xacro:property name="mesh_file" value="package://rotors_description/meshes/boreas.dae" />
-  <xacro:property name="mass" value="8.0" /> <!-- [kg] -->
+  <xacro:property name="mass" value="6.0" /> <!-- [kg] -->
   <xacro:property name="body_width" value="0.8378145" /> <!-- [m] -->
   <xacro:property name="body_height" value="0.510" /> <!-- [m] -->
@@ -18,4 +18,7 @@
   <xacro:property name="z_offset" value="0.024" /> <!-- [m] -->
   <xacro:property name="z_offset_direction" value="-0.0285" /> <!-- [m] -->
+  <xacro:property name="com_x" value="0.0" />
+  <xacro:property name="com_y" value="0.0" />
+  <xacro:property name="com_z" value="-0.0718471" />
   <xacro:property name="mass_rotor_thrust" value="0.05" /> <!-- [kg] -->
   <xacro:property name="mass_rotor_direction" value="0.01" /> <!-- [kg] -->
@@ -36,5 +39,5 @@
   <!-- Property Blocks -->
   <xacro:property name="body_inertia"> <!-- TODO -->
-    <inertia ixx="0.4559" ixy="0.0161" ixz="-0.0083" iyy="0.4489" iyz="0.0020" izz="0.6497" /> <!-- [kg.m^2] [kg.m^2] [kg.m^2] [kg.m^2] [kg.m^2] [kg.m^2] -->
+    <inertia ixx="0.4172" ixy="0.0165" ixz="-0.0085" iyy="0.4113" iyz="0.0022" izz="0.6498" /> <!-- [kg.m^2] [kg.m^2] [kg.m^2] [kg.m^2] [kg.m^2] [kg.m^2] -->
   </xacro:property>
     <!-- inertia of a single rotor, assuming it is a cuboid. Height=3mm, width=15mm -->
@@ -55,4 +58,7 @@
     use_mesh_file="${use_mesh_file}"
     mesh_file="${mesh_file}"
+    com_x="${com_x}"
+    com_y="${com_y}"
+    com_z="${com_z}"
     >
     <xacro:insert_block name="body_inertia" />

File: rotors_description/urdf/multirotor_base.xacro (robot description, xacro)
@@ -33,5 +33,5 @@
   <!-- Main multirotor link -->
   <xacro:macro name="multirotor_base_macro"
-    params="robot_namespace mass body_width body_height use_mesh_file mesh_file *inertia">
+    params="robot_namespace mass body_width body_height use_mesh_file mesh_file com_x com_y com_z *inertia" >
     <link name="${robot_namespace}/base_link"></link>
     <!-- origin -->
@@ -44,5 +44,5 @@
       <inertial>
         <mass value="${mass}" />  <!-- [kg] -->
-        <origin xyz="0 0 0" />
+        <origin xyz="${com_x} ${com_y} ${com_z}" rpy ="0 0 0" />
         <xacro:insert_block name="inertia" />
       </inertial>

Commit message: changes to boreas inertia

File: rotors_description/urdf/boreas.xacro (robot description, xacro)
@@ -7,15 +7,15 @@
   <xacro:property name="rotor_velocity_slowdown_sim" value="10" />
   <xacro:property name="use_mesh_file" value="true" />
-  <xacro:property name="mesh_file" value="package://rotors_description/meshes/boreas.dae" />
+  <xacro:property name="mesh_file" value="package://rotors_description/meshes/boreas_origin.dae" />
   <xacro:property name="mass" value="6.0" /> <!-- [kg] -->
   <xacro:property name="body_width" value="0.8378145" /> <!-- [m] -->
   <xacro:property name="body_height" value="0.510" /> <!-- [m] -->
-  <xacro:property name="auxiliary_x" value="0.452" /> <!-- [m] -->
-  <xacro:property name="auxiliary_y" value="0.452" /> <!-- [m] -->
+  <xacro:property name="auxiliary_x" value="0.455" /> <!-- [m] -->
+  <xacro:property name="auxiliary_y" value="0.455" /> <!-- [m] -->
   <xacro:property name="thrust_x" value="0.41890725" /> <!-- [m] -->
   <xacro:property name="thrust_y" value="0.41890725" /> <!-- [m] -->
   <xacro:property name="rotation" value="3.14" /> <!-- 180 degrees -->
-  <xacro:property name="z_offset" value="0.024" /> <!-- [m] -->
-  <xacro:property name="z_offset_direction" value="-0.0285" /> <!-- [m] -->
+  <xacro:property name="z_offset" value="0.0525" /> <!-- [m] -->
+  <xacro:property name="z_offset_direction" value="0.0" /> <!-- [m] -->
   <xacro:property name="com_x" value="0.0" />
   <xacro:property name="com_y" value="0.0" />

Commit message: corrected mass

File: rotors_description/urdf/boreas.xacro (robot description, xacro)
@@ -8,5 +8,5 @@
   <xacro:property name="use_mesh_file" value="true" />
   <xacro:property name="mesh_file" value="package://rotors_description/meshes/boreas_origin.dae" />
-  <xacro:property name="mass" value="6.0" /> <!-- [kg] -->
+  <xacro:property name="mass" value="7.5276" /> <!-- [kg] -->
   <xacro:property name="body_width" value="0.8378145" /> <!-- [m] -->
   <xacro:property name="body_height" value="0.510" /> <!-- [m] -->
