Commit message: boreas with one camera

File: rotors_description/urdf/boreas.xacro (robot description, xacro)
@@ -1,4 +1,4 @@
 <?xml version="1.0"?>
-<robot name="geranos" xmlns:xacro="http://ros.org/wiki/xacro">
+<robot name="$(arg mav_name)" xmlns:xacro="http://ros.org/wiki/xacro">
   <!-- Properties -->
   <xacro:property name="namespace" value="$(arg namespace)" />

File: rotors_description/urdf/boreas_base.xacro (robot description, xacro)
@@ -1,4 +1,4 @@
 <?xml version="1.0"?>
-<robot name="geranos" xmlns:xacro="http://ros.org/wiki/xacro">
+<robot name="$(arg mav_name)" xmlns:xacro="http://ros.org/wiki/xacro">
   <xacro:include filename="$(find rotors_description)/urdf/component_snippets.xacro" />
   <!-- Instantiate boreas "mechanics" -->
@@ -8,4 +8,65 @@
   <!-- Mount an ADIS16448 IMU. -->
   <xacro:default_imu namespace="${namespace}" parent_link="${namespace}/base_link" />
+ <!-- Manual ground truth odometry -->
+<!--   <xacro:odometry_plugin_macro
+    namespace="${namespace}"
+    odometry_sensor_suffix=""
+    parent_link="${namespace}/base_link"
+    pose_topic="pose"
+    pose_with_covariance_topic="pose_with_covariance"
+    position_topic="position"
+    transform_topic="transform"
+    odometry_topic="odometry"
+    parent_frame_id="world"
+    child_frame_id="${namespace}/base_link"
+    mass_odometry_sensor="0.00001"
+    measurement_divisor="1"
+    measurement_delay="0"
+    unknown_delay="0.0"
+    noise_normal_position="0 0 0"
+    noise_normal_quaternion="0 0 0"
+    noise_normal_linear_velocity="0 0 0"
+    noise_normal_angular_velocity="0 0 0"
+    noise_uniform_position="0 0 0"
+    noise_uniform_quaternion="0 0 0"
+    noise_uniform_linear_velocity="0 0 0"
+    noise_uniform_angular_velocity="0 0 0"
+    enable_odometry_map="false"
+    odometry_map=""
+    image_scale="">
+    <inertia ixx="0.00001" ixy="0.0" ixz="0.0" iyy="0.00001" iyz="0.0" izz="0.00001" />
+    <origin xyz="0.0 0.0 0.0" rpy="0.0 0.0 0.0" />
+  </xacro:odometry_plugin_macro> -->
+ <!-- odometry_sensor_rovio -> measurement_divisor has to be <= 3, but was 16 -->
+<!--   <xacro:odometry_plugin_macro
+  namespace="${namespace}"
+  odometry_sensor_suffix=""
+  parent_link="${namespace}/base_link"
+  pose_topic="pose"
+  pose_with_covariance_topic="pose_with_covariance"
+  position_topic="position"
+  transform_topic="transform"
+  odometry_topic="odometry"
+  parent_frame_id="world"
+  child_frame_id="${namespace}/base_link"
+  mass_odometry_sensor="0.00001"
+  measurement_divisor="1"
+  measurement_delay="0.002"
+  unknown_delay="0.0"
+  noise_normal_position="0.0075 0.01 0.003"
+  noise_normal_quaternion="0.0075 0.01 0.003"
+  noise_normal_linear_velocity="0.03 0.03 0.03"
+  noise_normal_angular_velocity="0.0075 0.01 0.003"
+  noise_uniform_position="0.001 0.001 0.001"
+  noise_uniform_quaternion="0.001 0.001 0.001"
+  noise_uniform_linear_velocity="0.001 0.001 0.001"
+  noise_uniform_angular_velocity="0.001 0.001 0.001"
+  enable_odometry_map="false"
+  odometry_map=""
+  image_scale="">
+  <inertia ixx="0.00001" ixy="0.0" ixz="0.0" iyy="0.00001" iyz="0.0" izz="0.00001" />
+  <origin xyz="0.0 0.0 0.0" rpy="0.0 0.0 0.0" />
+</xacro:odometry_plugin_macro> -->
+  <!-- <xacro:if value="false"> -->
   <xacro:if value="$(arg enable_ground_truth)">
     <xacro:ground_truth_imu_and_odometry namespace="${namespace}" parent_link="${namespace}/base_link" />
@@ -21,3 +82,45 @@
   <!-- Add odometry. -->
   <xacro:include filename="$(find mav_description)/urdf/odometry_sensor_rovio.xacro"/>
+  <!-- included directly odometry_sensor_rovio, changed measurement_divisor from 16 to 1 -->
+<!--   <robot name="$(arg mav_name)" xmlns:xacro="http://ros.org/wiki/xacro">
+    <xacro:odometry_plugin_macro
+      namespace="${namespace}"
+      odometry_sensor_suffix="1"
+      parent_link="${namespace}/base_link"
+      pose_topic="odometry_sensor1/pose"
+      pose_with_covariance_topic="odometry_sensor1/pose_with_covariance"
+      position_topic="odometry_sensor1/position"
+      transform_topic="odometry_sensor1/transform"
+      odometry_topic="odometry_sensor1/odometry"
+      parent_frame_id="world"
+      child_frame_id="${namespace}/odometry_sensor1"
+      mass_odometry_sensor="0.00001"
+      measurement_divisor="1"
+      measurement_delay="0.002"
+      unknown_delay="0.0"
+      noise_normal_position="0.0075 0.01 0.003"
+      noise_normal_quaternion="0.0075 0.01 0.003"
+      noise_normal_linear_velocity="0.03 0.03 0.03"
+      noise_normal_angular_velocity="0.0075 0.01 0.003"
+      noise_uniform_position="0.001 0.001 0.001"
+      noise_uniform_quaternion="0.001 0.001 0.001"
+      noise_uniform_linear_velocity="0.001 0.001 0.001"
+      noise_uniform_angular_velocity="0.001 0.001 0.001"
+      enable_odometry_map="false"
+      odometry_map=""
+      image_scale="">
+      <inertia ixx="0.00001" ixy="0.0" ixz="0.0" iyy="0.00001" iyz="0.0" izz="0.00001" />
+      <origin xyz="0.0 0.0 0.0" rpy="0.0 0.0 0.0" />
+    </xacro:odometry_plugin_macro>
+  </robot> -->
+              <!-- [kg m^2] [kg m^2] [kg m^2] [kg m^2] [kg m^2] [kg m^2] -->
+    <!-- Add realsense -->
+  <xacro:if value="$(arg add_rgbd_sensor)">
+    <!-- Import macro for realsense-RS200 camera-->
+    <xacro:include filename="$(find realsense_gazebo_plugin)/urdf/realsense-D435.macro.xacro"/>
+    <!-- Create camera instance -->
+    <xacro:realsense-D435 prefix="" parent="${namespace}/base_link">
+        <origin xyz="0.18 0.0 -0.2565" rpy="0.0 ${-10.0/180.0*pi} 0.0" />
+    </xacro:realsense-D435>
+  </xacro:if>
 </robot>

Commit message: easy xarco

File: rotors_description/urdf/boreas.xacro (robot description, xacro)
@@ -8,5 +8,5 @@
   <xacro:property name="use_mesh_file" value="true" />
   <xacro:property name="mesh_file" value="package://rotors_description/meshes/boreas_origin.dae" />
-  <xacro:property name="mass" value="7.5276" /> <!-- [kg] -->
+  <xacro:property name="mass" value="7" /> <!-- 7.5276[kg] -->
   <xacro:property name="body_width" value="0.8378145" /> <!-- [m] -->
   <xacro:property name="body_height" value="0.510" /> <!-- [m] -->
@@ -20,5 +20,6 @@
   <xacro:property name="com_x" value="0.0" />
   <xacro:property name="com_y" value="0.0" />
-  <xacro:property name="com_z" value="-0.0718471" />
+  <xacro:property name="com_z" value="-0.0718471" /> <!-- center of mass offset -->
+  <!-- <xacro:property name="com_z" value="-0.0718471" /> -->
   <xacro:property name="mass_rotor_thrust" value="0.05" /> <!-- [kg] -->
   <xacro:property name="mass_rotor_direction" value="0.01" /> <!-- [kg] -->
@@ -39,5 +40,7 @@
   <!-- Property Blocks -->
   <xacro:property name="body_inertia"> <!-- TODO -->
-    <inertia ixx="0.4172" ixy="0.0165" ixz="-0.0085" iyy="0.4113" iyz="0.0022" izz="0.6498" /> <!-- [kg.m^2] [kg.m^2] [kg.m^2] [kg.m^2] [kg.m^2] [kg.m^2] -->
+    <inertia ixx="0.5" ixy="0.0" ixz="0.0" iyy="0.5" iyz="0.0" izz="0.7" />
+<!--     <inertia ixx="0.4172" ixy="0.0165" ixz="-0.0085" iyy="0.4113" iyz="0.0022" izz="0.6498" /> -->
+     <!--  [kg.m^2] [kg.m^2] [kg.m^2] [kg.m^2] [kg.m^2] [kg.m^2] -->
   </xacro:property>
     <!-- inertia of a single rotor, assuming it is a cuboid. Height=3mm, width=15mm -->

Commit message: com update

File: rotors_description/urdf/boreas.xacro (robot description, xacro)
@@ -20,5 +20,5 @@
   <xacro:property name="com_x" value="0.0" />
   <xacro:property name="com_y" value="0.0" />
-  <xacro:property name="com_z" value="-0.0718471" /> <!-- center of mass offset -->
+  <xacro:property name="com_z" value="-0.07" /> <!-- center of mass offset -->
   <!-- <xacro:property name="com_z" value="-0.0718471" /> -->
   <xacro:property name="mass_rotor_thrust" value="0.05" /> <!-- [kg] -->
