Commit message: added second realsense

File: rotors_description/urdf/boreas_base.xacro (robot description, xacro)
@@ -119,7 +119,11 @@
     <!-- Import macro for realsense-RS200 camera-->
     <xacro:include filename="$(find realsense_gazebo_plugin)/urdf/realsense-D435.macro.xacro"/>
-    <!-- Create camera instance -->
-    <xacro:realsense-D435 prefix="" parent="${namespace}/base_link">
+    <!-- Create camera instance 1-->
+    <xacro:realsense-D435 prefix="/boreas/camera/left/" parent="${namespace}/base_link">
         <origin xyz="0.18 0.0 -0.2565" rpy="0.0 ${-10.0/180.0*pi} 0.0" />
+    </xacro:realsense-D435>
+    <!-- Create camera instance 1-->
+    <xacro:realsense-D435 prefix="/boreas/camera/right/" parent="${namespace}/base_link">
+        <origin xyz="0.18 0.0 -0.2" rpy="0.0 ${0.0/180.0*pi} 0.0" />
     </xacro:realsense-D435>
   </xacro:if>

Commit message: two realsenses top bottom horizontal

File: rotors_description/urdf/boreas_base.xacro (robot description, xacro)
@@ -120,10 +120,10 @@
     <xacro:include filename="$(find realsense_gazebo_plugin)/urdf/realsense-D435.macro.xacro"/>
     <!-- Create camera instance 1-->
-    <xacro:realsense-D435 prefix="/boreas/camera/left/" parent="${namespace}/base_link">
-        <origin xyz="0.18 0.0 -0.2565" rpy="0.0 ${-10.0/180.0*pi} 0.0" />
+    <xacro:realsense-D435 prefix="boreas/camera/left/" parent="${namespace}/base_link">
+        <origin xyz="0.18 0.0 -0.2565" rpy="0.0 ${-15.0/180.0*pi} 0.0" />
     </xacro:realsense-D435>
-    <!-- Create camera instance 1-->
-    <xacro:realsense-D435 prefix="/boreas/camera/right/" parent="${namespace}/base_link">
-        <origin xyz="0.18 0.0 -0.2" rpy="0.0 ${0.0/180.0*pi} 0.0" />
+    <!-- Create camera instance 2-->
+    <xacro:realsense-D435 prefix="boreas/camera/right/" parent="${namespace}/base_link">
+        <origin xyz="0.18 0.0 -0.05" rpy="0 ${10.0/180.0*pi} ${0/180.0*pi}" />
     </xacro:realsense-D435>
   </xacro:if>

Commit message: improve camera angle

File: rotors_description/urdf/boreas_base.xacro (robot description, xacro)
@@ -125,5 +125,5 @@
     <!-- Create camera instance 2-->
     <xacro:realsense-D435 prefix="boreas/camera/right/" parent="${namespace}/base_link">
-        <origin xyz="0.18 0.0 -0.05" rpy="0 ${10.0/180.0*pi} ${0/180.0*pi}" />
+        <origin xyz="0.18 0.0 -0.05" rpy="0 ${5.0/180.0*pi} ${0/180.0*pi}" />
     </xacro:realsense-D435>
   </xacro:if>

Commit message: less camera overlap, renaming to top/bottom

File: rotors_description/urdf/boreas_base.xacro (robot description, xacro)
@@ -120,10 +120,10 @@
     <xacro:include filename="$(find realsense_gazebo_plugin)/urdf/realsense-D435.macro.xacro"/>
     <!-- Create camera instance 1-->
-    <xacro:realsense-D435 prefix="boreas/camera/left/" parent="${namespace}/base_link">
+    <xacro:realsense-D435 prefix="boreas/camera/bottom/" parent="${namespace}/base_link">
         <origin xyz="0.18 0.0 -0.2565" rpy="0.0 ${-15.0/180.0*pi} 0.0" />
     </xacro:realsense-D435>
     <!-- Create camera instance 2-->
-    <xacro:realsense-D435 prefix="boreas/camera/right/" parent="${namespace}/base_link">
-        <origin xyz="0.18 0.0 -0.05" rpy="0 ${5.0/180.0*pi} ${0/180.0*pi}" />
+    <xacro:realsense-D435 prefix="boreas/camera/top/" parent="${namespace}/base_link">
+        <origin xyz="0.18 0.0 -0.15" rpy="0 ${10.0/180.0*pi} ${0/180.0*pi}" />
     </xacro:realsense-D435>
   </xacro:if>

Commit message: added realsense camera

File: rotors_description/urdf/boreas_base.xacro (robot description, xacro)
@@ -4,4 +4,13 @@
   <!-- Instantiate boreas "mechanics" -->
   <xacro:include filename="$(find rotors_description)/urdf/boreas.xacro" />
+      <!-- Add realsense -->
+  <xacro:if value="$(arg add_rgbd_sensor)">
+    <!-- Import macro for realsense-RS200 camera-->
+    <xacro:include filename="$(find realsense_gazebo_plugin)/urdf/realsense-D435.macro.xacro"/>
+    <!-- Create camera instance -->
+    <xacro:realsense-D435 prefix="" parent="${namespace}/base_link">
+        <origin xyz="0.18 0.0 -0.15" rpy="0.0 ${10.0/180.0*pi} 0.0" />
+    </xacro:realsense-D435>
+  </xacro:if>
   <!-- Instantiate a controller. -->
   <xacro:controller_plugin_macro namespace="${namespace}" imu_sub_topic="imu" />

Commit message: top 15 deg

File: rotors_description/urdf/boreas_base.xacro (robot description, xacro)
@@ -125,5 +125,5 @@
     <!-- Create camera instance 2-->
     <xacro:realsense-D435 prefix="boreas/camera/top/" parent="${namespace}/base_link">
-        <origin xyz="0.18 0.0 -0.15" rpy="0 ${10.0/180.0*pi} ${0/180.0*pi}" />
+        <origin xyz="0.18 0.0 -0.15" rpy="0 ${15.0/180.0*pi} ${0/180.0*pi}" />
     </xacro:realsense-D435>
   </xacro:if>
